File: PCB_ESP32_CAN/PCB_ESP32_CAN.kicad_sch (KiCad schematic)
At the start: 53 parts, among them J1 USB_C_Receptacle_USB2.0, J2 CAN, J3 CAN, J4 CAN, J5 CAN, Q1 Q_NPN_BCE, Q2 Q_NPN_BCE, SW1 RST, SW2 BOOT, U1 ESP32-WROOM-32, U2 CP2102N-A01-GQFN24, U3 SN65HVD232, U4 NCP1117-3.3_SOT223

Commit message: V2.0 ESP32 pcb
Parts:
- removed J4, J5: CAN, AREA_lib_Connector:Wuerth_2mm_4pin_62000411622, symbol Connector:Conn_01x04_Male
- removed R1, R6: 560, Resistor_SMD:R_0805_2012Metric_Pad1.20x1.40mm_HandSolder, symbol Device:R
- removed R5: 10K, Resistor_SMD:R_0805_2012Metric_Pad1.20x1.40mm_HandSolder, symbol Device:R
- added C16: 10u, Capacitor_SMD:C_0805_2012Metric_Pad1.18x1.45mm_HandSolder, symbol Device:C
- added R16: 47k5, Resistor_SMD:R_0805_2012Metric_Pad1.20x1.40mm_HandSolder, symbol Device:R
- added R17: 10k, Resistor_SMD:R_0805_2012Metric_Pad1.20x1.40mm_HandSolder, symbol Device:R
- added TP1: RTS, TestPoint:TestPoint_Pad_D1.0mm, symbol Connector:TestPoint
- added TP2: DTR, TestPoint:TestPoint_Pad_D1.0mm, symbol Connector:TestPoint
- added TP3: RX, TestPoint:TestPoint_Pad_D1.0mm, symbol Connector:TestPoint
- added TP4: TX, TestPoint:TestPoint_Pad_D1.0mm, symbol Connector:TestPoint
- added TP5: CANH, TestPoint:TestPoint_THTPad_D2.0mm_Drill1.0mm, symbol Connector:TestPoint
- added TP6: CANL, TestPoint:TestPoint_THTPad_D2.0mm_Drill1.0mm, symbol Connector:TestPoint
- C1, C12, C2: value 1n -> 100n
- R10: value 260 -> 270
- R7: value 10K -> 22k1
Connections:
- net +3V3: now also C16.1, R17.1; no longer D1.2 (A), D2.2 (A), R7.1, U2.5 (VIO)
- net +5V: now also R7.1; no longer U2.8 (VBUS)
- net CANH: now also TP5.1
- net CANL: now also TP6.1
- net DTR: now also TP2.1
- net EN: now also C1.1, SW1.2
- net GND: now also D1.1 (K), D2.1 (K), SW1.1, C16.2, R16.2; no longer SW1.2
- net IO0: now also C12.1, SW2.1
- net RTS: now also TP1.1
- net RX: now also TP3.1
- net TX: now also TP4.1
- net at R7.2: now also U2.8 (VBUS), R16.1; no longer U2.9 (~{RSTb})
- net at R9.1: now also D1.2 (A); no longer D1.1 (K)
- net at R10.1: now also D2.2 (A); no longer D2.1 (K)
- new net: R17.2, U2.9 (~{RSTb})
- no-connect marks 10 -> 11
Other:
- note removed: "PAS BON"
- moved on the sheet: C1, C11, C2, C9, D1, D2, R10, R8, R9, SW1

Commit message: Maj carte alim
Other:
- note added: "Autoprogram"
- note added: "CANbus"
- note added: "NC"
- note added: "Power supply 5V/3V3"
- note added: "USB to UART"
- moved on the sheet: C1, C12, C13, C14, C15, C16, C2, C3, C5, D1, D2, D3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

Commit message: update
Parts:
- C1, C10, C11, C12, C13, C14, C15, C16, C2, C3, C4, C5, C6, C7, C8, C9: footprint Capacitor_SMD:C_0805_2012Metric_Pad1.18x1.45mm_HandSolder -> Capacitor_SMD:C_0805_2012Metric
- D1, D2, D3, D4: footprint LED_SMD:LED_0805_2012Metric_Pad1.15x1.40mm_HandSolder -> LED_SMD:LED_0805_2012Metric
- Q1, Q2: value Q_NPN_BCE -> MMBT2222ALT1G; symbol Device:Q_NPN_BCE -> Device:Q_NPN_BEC
- R10, R11, R12, R13, R14, R15, R16, R17, R2, R3, R4, R7, R8, R9: footprint Resistor_SMD:R_0805_2012Metric_Pad1.20x1.40mm_HandSolder -> Resistor_SMD:R_0805_2012Metric
- TP5, TP6: footprint TestPoint:TestPoint_THTPad_D2.0mm_Drill1.0mm -> TestPoint:TestPoint_Pad_D1.0mm
Connections:
- net +3V3: now also D1.1 (K), D2.1 (K)
- net DTR: now also Q2.2 (E); no longer Q2.3 (E)
- net EN: now also Q1.3 (C); no longer Q1.2 (C)
- net GND: no longer D1.1 (K), D2.1 (K)
- net IO0: now also Q2.3 (C); no longer Q2.2 (C)
- net RTS: now also Q1.2 (E); no longer Q1.3 (E)
Other:
- moved on the sheet: D2, R10
