File: PCB_Pompe_V2/PCB_Pompe_V2.sch (KiCad schematic (older format))
At the start: 34 parts, among them J1 Conn_01x04_Female, J13 Conn_01x05_Female, J2 Conn_01x04_Female, J8 Conn_01x02_Male, SW1 SW_Push, U1 SN65HVD232, U2 STM32F302C6Tx, U3 NCP1117-3.3_SOT223, Y1 8MHz

Commit message: IO prete, Pompe finir sérigraphie, Alim+AX12 à faire
Parts:
- Y1: symbol Device:Crystal_GND23_Small -> Device:Crystal_GND24_Small
Connections:
- net V14 is gone; now on net P8: U2.38 (PA15)
- net GND: now also Y1.4; no longer Y1.3
- net P5: now also U2.18 (PB0); no longer U2.29 (PA8)
- net P6: now also U2.29 (PA8); no longer U2.31 (PA10)
- net P7: now also U2.31 (PA10); no longer U2.18 (PB0)
- net P8: no longer U2.20 (PB2)
- net V5: now also U2.19 (PB1); no longer U2.30 (PA9)
- net V6: now also U2.30 (PA9); no longer U2.32 (PA11)
- net V7: now also U2.32 (PA11); no longer U2.19 (PB1)
- net at C2.1, U2.6 (PF1): now also Y1.3; no longer Y1.4
- net P11: no longer names the net of U2.21 (PB10)
- net P12: no longer names the net of U2.25 (PB12)
- net P14: no longer names the net of U2.33 (PA12)
- net P15: no longer names the net of U2.27 (PB14)
- net V11: no longer names the net of U2.22 (PB11)
- net V12: no longer names the net of U2.26 (PB13)
- no-connect marks 1 -> 2
Changed lines of the file:
@@
 $Descr A4 11693 8268
 encoding utf-8
-Sheet 1 16
+Sheet 1 11
 Title "PCB Pompe"
 Date ""
@@
 SWCLK
 $Comp
-L Device:Crystal_GND23_Small Y1
+L Device:Crystal_GND24_Small Y1
 U 1 1 5FB44954
 P 950 1400
@@
 Text GLabel 2600 2650 2    50   Input ~ 0
 P4
-Text GLabel 2600 2850 2    50   Input ~ 0
+Text GLabel 1300 2050 0    50   Input ~ 0
 P5
-Text GLabel 1300 2250 0    50   Input ~ 0
+Text GLabel 2600 3550 2    50   Input ~ 0
 P8
 Text GLabel 2600 2150 2    50   Input ~ 0
@@
 Text GLabel 2600 2350 2    50   Input ~ 0
 V2
-Text GLabel 1300 2150 0    50   Input ~ 0
+Text GLabel 2600 3150 2    50   Input ~ 0
 V7
 Text GLabel 1300 2450 0    50   Input ~ 0
@@
 Text GLabel 2600 2750 2    50   Input ~ 0
 V4
-Text GLabel 2600 2950 2    50   Input ~ 0
+Text GLabel 1300 2150 0    50   Input ~ 0
 V5
 Text GLabel 1300 2350 0    50   Input ~ 0
@@
 Text GLabel 1300 2550 0    50   Input ~ 0
 V9
-Text GLabel 2600 3050 2    50   Input ~ 0
+Text GLabel 2600 2850 2    50   Input ~ 0
 P6
-Text GLabel 2600 3150 2    50   Input ~ 0
+Text GLabel 2600 2950 2    50   Input ~ 0
 V6
 $Comp
@@
 Wire Wire Line
 	1800 3750 1900 3750
-Text GLabel 1300 2050 0    50   Input ~ 0
+Text GLabel 2600 3050 2    50   Input ~ 0
 P7
 Wire Wire Line
@@
 Text GLabel 1300 2750 0    50   Input ~ 0
 V10
-Text GLabel 1300 3050 0    50   Input ~ 0
-P11
-Text GLabel 1300 3150 0    50   Input ~ 0
-V11
-Text GLabel 1300 3250 0    50   Input ~ 0
-P12
-Text GLabel 1300 3350 0    50   Input ~ 0
-V12
 Text GLabel 1300 1650 0    50   Input ~ 0
 P13
 Text GLabel 1300 1750 0    50   Input ~ 0
 V13
-Text GLabel 2600 3250 2    50   Input ~ 0
-P14
-Text GLabel 2600 3550 2    50   Input ~ 0
-V14
-Text GLabel 1300 3450 0    50   Input ~ 0
-P15
 Text GLabel 1300 1850 0    50   Input ~ 0
 V15
@@
 F1 "MOS10.sch" 50
 $EndSheet
-$Sheet
-S 5850 3650 650  400
-U 61AB277D
-F0 "sheet61AB2776" 50
-F1 "MOS11.sch" 50
-$EndSheet
-$Sheet
-S 6750 3650 650  400
-U 61AB277F
-F0 "sheet61AB2777" 50
-F1 "MOS12.sch" 50
-$EndSheet
-$Sheet
-S 4100 4250 650  400
-U 61AB9540
-F0 "sheet61AB953B" 50
-F1 "MOS13.sch" 50
-$EndSheet
-$Sheet
-S 5000 4250 650  400
-U 61AB9542
-F0 "sheet61AB953C" 50
-F1 "MOS14.sch" 50
-$EndSheet
-$Sheet
-S 5850 4250 650  400
-U 61AB9544
-F0 "sheet61AB953D" 50
-F1 "MOS15.sch" 50
-$EndSheet
+NoConn ~ 950  1700
 $EndSCHEMATC
