File: PCB_Pompe_V2/PCB_Pompe_V2.kicad_pcb (KiCad board)
At the start: 2 copper layers, 87.5 x 52.5 mm, 142 parts, among them J1 Conn_01x04_Female, J10 Conn_01x03_Female, J11 Conn_01x03_Female, J12 Conn_01x03_Female, J13 Conn_01x05_Female, J14 Conn_01x03_Female, J2 Conn_01x04_Female, J3 Conn_01x03_Female, J4 Conn_01x03_Female, J5 Conn_01x03_Female, J6 Conn_01x03_Female, J7 Conn_01x03_Female, J8 Conn_01x02_Male, J9 Conn_01x03_Female, Q1 DMN10H700S, Q10 DMN10H700S, Q11 DMN10H700S, Q12 DMN10H700S, Q13 DMN10H700S, Q14 DMN10H700S, Q15 DMN10H700S, Q16 DMN10H700S, Q17 DMN10H700S, Q18 DMN10H700S, Q19 DMN10H700S, Q2 DMN10H700S, Q20 DMN10H700S, Q3 DMN10H700S, Q4 DMN10H700S, Q5 DMN10H700S, Q6 DMN10H700S, Q7 DMN10H700S, Q8 DMN10H700S, Q9 DMN10H700S, U1 SN65HVD232, U2 STM32F302C6Tx, U3 NCP1117-3.3_SOT223, Y1 8MHz

Commit message: lots of stuf
Routing:
- net +3V3: track 95.4 -> 94.1 mm
- net CANL: track 46.5 -> 47.5 mm
- net CANH: track 41.3 -> 42.3 mm
- net +5V: track 41.5 -> 40.9 mm
- net GND: vias 77 -> 74
Other:
- net class Default removed
- board text added: "."
- board text added: "3V3"
- board text added: "5V"
- board text added: "CLK"
- board text added: "GND"
- board text added: "IO"
- board text added: "P1 V1"
- board text added: "P10 V10"
- board text added: "P2 V2"
- board text added: "P3 V3"
- board text added: "P4 V4"
- board text added: "P5 V5"
- board text added: "P6 V6"
- board text added: "P7 V7"
- board text added: "P8 V8"
- board text added: "P9 V9"
- board text added: "RST"
