File: IO_Board_V1/IO_Board_V1.sch (KiCad schematic (older format))
At the start: 92 parts, among them J1 USB_C_Receptacle_USB2.0, J10 IFM1, J11 FOURCHE, J12 BTN, J13 FOURCHE, J14 BTN, J15 CON_UART, J16 BTN, J17 FOURCHE, J18 IFM2, J19 IFM3, J2 CON_debug, J20 FOURCHE, J21 CON_I2C, J22 IFM4, J23 SPI, J24 BTN, J3 Conn_ARM_JTAG_SWD_10, J4 CON_CAN, J5 CON_CAN, J6 12V, J7 BTN, J8 BTN, J9 IFM0, SW1 BOOT, SW2 RST, U1 STM32F302C6Tx, U2 NCP1117-3.3_SOT223, U3 SN65HVD232, Y1 8MHz

Commit message: new alim pcb
Parts:
- J1: symbol Connector:USB_C_Receptacle_USB2.0 -> IO_Board_V1-rescue:USB_C_Receptacle_USB2.0-Connector
Changed lines of the file:
@@
 	10100 5550 10000 5550
 $Comp
-L Connector:USB_C_Receptacle_USB2.0 J1
+L IO_Board_V1-rescue:USB_C_Receptacle_USB2.0-Connector J1
 U 1 1 61685184
 P 5150 2000
