File: IO_Board_V1/IO_Board_V1.kicad_pcb (KiCad board)
At the start: 2 copper layers, 78 x 48 mm, 92 parts, among them J1 USB_C_Receptacle_USB2.0, J10 IFM1, J11 FOURCHE, J12 BTN, J13 FOURCHE, J14 BTN, J15 CON_UART, J16 BTN, J17 FOURCHE, J18 IFM2, J19 IFM3, J2 CON_debug, J20 FOURCHE, J21 CON_I2C, J22 IFM4, J23 SPI, J24 BTN, J3 Conn_ARM_JTAG_SWD_10, J4 CON_CAN, J5 CON_CAN, J6 12V, J7 BTN, J8 BTN, J9 IFM0, U1 STM32F302C6Tx, U2 NCP1117-3.3_SOT223, U3 SN65HVD232, Y1 8MHz

Commit message: new alim pcb
Parts:
- moved CANL1 0.84 mm to (94.8, 121.7)

Commit message: some changes
Other:
- board text added: "IFM0"

Commit message: lots of stuf
Parts:
- R3: value 270 -> 560
- renumbered 120 to JP1, BOOT to SW1, RST to SW2
Connections:
- J1 pad A8: Net-(J1-PadA8) -> unconnected-(J1-PadA8)
- J1 pad B8: Net-(J1-PadB8) -> unconnected-(J1-PadB8)
- J3 pad 4: /CLK -> /SWCLK
- J3 pad 7: Net-(J3-Pad7) -> unconnected-(J3-Pad7)
- J3 pad 8: Net-(J3-Pad8) -> unconnected-(J3-Pad8)
- U1 pad 1: Net-(U1-Pad1) -> unconnected-(U1-Pad1)
- U1 pad 2: Net-(U1-Pad2) -> unconnected-(U1-Pad2)
- U1 pad 3: Net-(U1-Pad3) -> unconnected-(U1-Pad3)
- U1 pad 4: Net-(U1-Pad4) -> unconnected-(U1-Pad4)
- U3 pad 5: Net-(U3-Pad5) -> unconnected-(U3-Pad5)
- U3 pad 8: Net-(U3-Pad8) -> unconnected-(U3-Pad8)
Other:
- net class Default removed
