File: Carte_Alim_V5/Carte_Alim_V5.sch (KiCad schematic (older format))
At the start: 46 parts, among them J1 BAT_IN, J10 12VC, J11 12VC, J12 12VC, J13 12VP, J14 12VP, J15 12VP, J16 12VP, J17 12VP, J18 12VP, J19 5VC, J2 BAT_IN, J20 5V_CAN, J21 5VC, J22 5V_CAN, J23 5VC, J24 5V_CAN, J25 5VC, J26 5V_CAN, J27 5VP, J28 5VP, J29 5VP, J3 MOT_OUT, J30 5VP, J31 5VP, J32 5VP, J4 MOT_OUT, J5 MOT_OUT, J6 MOT_OUT, J7 12VC, J8 12VC, J9 12VC

Commit message: new alim pcb
Parts:
- removed C10, C11, C13: 10u, Capacitor_THT:CP_Radial_D4.0mm_P2.00mm, symbol Device:CP_Small
- removed C12, C14, C15: 47u, Capacitor_THT:CP_Radial_D4.0mm_P2.00mm, symbol Device:CP_Small
- removed F1: 3557-2, AREA_lib_composant:FUSE_3557-2, symbol AREA_composant:3557-2
- removed J10, J11, J12, J7, J8, J9: 12VC, AREA_lib_Connector:Wuerth_2.54mm_2pins_61900211121, symbol Connector:Conn_01x02_Male
- removed J13, J14, J15, J16, J17, J18: 12VP, AREA_lib_Connector:Wuerth_3.96mm_2pin_645002114822, symbol Connector:Conn_01x02_Male
- removed J19, J21, J23, J25: 5VC, AREA_lib_Connector:Wuerth_2.54mm_2pins_61900211121, symbol Connector:Conn_01x02_Male
- removed J20, J22, J24, J26: 5V_CAN, AREA_lib_Connector:690367290476, symbol Connector:Conn_01x04_Male
- removed J27, J28, J29, J30, J31, J32: 5VP, AREA_lib_Connector:Wuerth_3.96mm_2pin_645002114822, symbol Connector:Conn_01x02_Male
- removed J3, J4, J5, J6: MOT_OUT, AREA_lib_Connector:Wuerth_batcon_691313710002, symbol Connector:Conn_01x02_Male
- removed PS1, PS2, PS3: TSR_2-2450, AREA_lib_composant:CONV_TSR_2-2450, symbol AREA_composant:TSR_2-2450
- added C? (x2): 47u, symbol Device:CP
- added C? (x8): 22u, symbol Device:C
- added C?: 4.7u, symbol Device:C
- added C?: 1u, symbol Device:C
- added C?: 0.1u, symbol Device:C
- added D?: LED, symbol Device:LED
- added L?: L, symbol Device:L
- added R? (x3): 10k, symbol Device:R
- added R? (x3): 8.87k, symbol Device:R
- added R?: 3.3, symbol Device:R
- added U?: SIC453, symbol AREA_composant:SIC453
Connections:
- net labels added: EN, PGOOD, PULLUP_VTG, SALERT, SCL, SDA, VDD, VOUT
- net labels removed: +12C, +12P, +24V, +5C, +5P, +5V
- wire segments 109 -> 97
- no-connect marks 8 -> 3
Other:
- note removed: "Convertisseur Buck 12V 5A"
- note removed: "Sortie 12V/3A commande"
- note removed: "Sortie 12V/5A puissance"
- note removed: "Sortie 5V/3A commande + CAN"
- note removed: "Sortie 5V/5A puissance"
- note removed: "Sortie stepper direct batterie"
- moved on the sheet: J2

Commit message: finalizing routing for test pcb buck
Parts:
- removed C? (x2): 47u, symbol Device:CP
- removed C? (x2): 22u, symbol Device:C
- removed C?: 4.7u, symbol Device:C
- removed C?: 1u, symbol Device:C
- removed R? (x2): 10k, symbol Device:R
- removed R? (x3): 8.87k, symbol Device:R
- removed U?: SIC453, symbol AREA_composant:SIC453
- added C1, C12, C19: 100n, Capacitor_SMD:C_0805_2012Metric_Pad1.15x1.40mm_HandSolder, symbol Device:C
- added C10, C11: 1u, Capacitor_SMD:C_0805_2012Metric_Pad1.15x1.40mm_HandSolder, symbol Device:C
- added C13, C14, C15, C16, C17, C18: 22u, Capacitor_SMD:C_1210_3225Metric_Pad1.42x2.65mm_HandSolder, symbol Device:C
- added C8: 33n, Capacitor_SMD:C_0805_2012Metric_Pad1.15x1.40mm_HandSolder, symbol Device:C
- added R2: 2k, Resistor_SMD:R_0603_1608Metric_Pad1.05x0.95mm_HandSolder, symbol Device:R
- added R3: 562k, Resistor_SMD:R_0603_1608Metric_Pad1.05x0.95mm_HandSolder, symbol Device:R
- added R4: 226k, Resistor_SMD:R_0603_1608Metric_Pad1.05x0.95mm_HandSolder, symbol Device:R
- added R5: 88.7k, Resistor_SMD:R_0603_1608Metric_Pad1.05x0.95mm_HandSolder, symbol Device:R
- added R6: 100k, Resistor_SMD:R_0603_1608Metric_Pad1.05x0.95mm_HandSolder, symbol Device:R
- added R8: 52.3k, Resistor_SMD:R_0603_1608Metric_Pad1.05x0.95mm_HandSolder, symbol Device:R
- added R9: 10k, Resistor_SMD:R_0603_1608Metric_Pad1.05x0.95mm_HandSolder, symbol Device:R
- added U1: SIC466ED-T1-GE3, AREA_lib_composant:CONV_SIC461ED-T1-GE3, symbol AREA_composant:SIC461ED-T1-GE3
- C2, C3, C4, C5, C6, C7: renamed from C?; footprint (none) -> Capacitor_SMD:C_1210_3225Metric_Pad1.42x2.65mm_HandSolder
- C9: renamed from C?; value 0.1u -> 100n; footprint (none) -> Capacitor_SMD:C_0805_2012Metric_Pad1.15x1.40mm_HandSolder
- D1: renamed from D?; footprint (none) -> LED_SMD:LED_0805_2012Metric_Pad1.15x1.40mm_HandSolder
- L1: renamed from L?; value L -> 4.7uH; footprint (none) -> Inductor_SMD:L_Vishay_IHLP-6767
- R1, R7: renamed from R?; footprint (none) -> Resistor_SMD:R_0603_1608Metric_Pad1.05x0.95mm_HandSolder
Connections:
- net +BATT: now also C1.1, C19.1, R3.1, U1.1 (VCIN), U1.29 (VIN), U1.7 (VIN), U1.8 (VIN)
- net GND: now also D1.1 (K), C1.2, C10.1, C11.1, C12.2, C13.2, C14.2, C15.2, C16.2, C17.2, C18.2, C19.2, C8.2, R2.2, R4.2, R5.2, R9.1, U1.10 (PGND), U1.11 (PGND), U1.17 (PGND), U1.23 (AGND), U1.28 (AGND), U1.30.1 (PGND), U1.30.2 (PGND), U1.9 (PGND)
- net VDD: now also C11.2, R6.1, U1.25 (ILIMIT), U1.26 (VDD)
- net VOUT: now also L1.2, C12.1, C13.1, C14.1, C15.1, C16.1, C17.1, C18.1, R8.2, U1.20 (VSNS)
- net at R7.1: now also U1.4 (BOOT)
- net at C9.2: now also U1.5 (PHASE), U1.6 (PHASE)
- net at L1.1: now also U1.12 (SW), U1.13 (SW), U1.14 (SW), U1.14.1 (SW)
- new net: C10.2, U1.16 (VDRV)
- new net: C8.1, U1.19 (SS)
- new net: R6.2, U1.2 (PGOOD)
- new net: R8.1, R9.2, U1.22 (VFB)
- new net: R5.1, U1.24 (FSW)
- new net: R2.1, U1.27 (MODE)
- new net: R3.2, R4.1, U1.3 (EN)
Other:
- note added: "1210\n"
- note added: "IHLP6767GZER4R7M11"
- note added: "close to Vcin"
- moved on the sheet: C9, L1, R7

Commit message: last version of alim v5
Parts:
- added D2: LED, LED_SMD:LED_0805_2012Metric_Pad1.15x1.40mm_HandSolder, symbol Device:LED
- added R10: 10k, Resistor_SMD:R_0603_1608Metric_Pad0.98x0.95mm_HandSolder, symbol Device:R
- J1, J2: footprint AREA_lib_Connector:Wuerth_batcon_691313710002 -> Connector_Phoenix_MSTB:PhoenixContact_MSTBVA_2,5_2-G-5,08_1x02_P5.08mm_Vertical
- U1: symbol AREA_composant:SIC461ED-T1-GE3 -> Carte_Alim_V5-rescue:SIC461ED-T1-GE3-AREA_composant
Connections:
- net GND: now also D2.1 (K)
- net VOUT: now also R10.1
- new net: D2.2 (A), R10.2
Changed lines of the file:
@@
 F 0 "J2" H 2158 1131 50  0000 C CNN
 F 1 "BAT_IN" H 2158 1040 50  0000 C CNN
-F 2 "AREA_lib_Connector:Wuerth_batcon_691313710002" H 2050 950 50  0001 C CNN
+F 2 "Connector_Phoenix_MSTB:PhoenixContact_MSTBVA_2,5_2-G-5,08_1x02_P5.08mm_Vertical" H 2050 950 50  0001 C CNN
 F 3 "~" H 2050 950 50  0001 C CNN
 	1    2050 950
@@
 F 0 "J1" H 1208 1131 50  0000 C CNN
 F 1 "BAT_IN" H 1208 1040 50  0000 C CNN
-F 2 "AREA_lib_Connector:Wuerth_batcon_691313710002" H 1100 950 50  0001 C CNN
+F 2 "Connector_Phoenix_MSTB:PhoenixContact_MSTBVA_2,5_2-G-5,08_1x02_P5.08mm_Vertical" H 1100 950 50  0001 C CNN
 F 3 "~" H 1100 950 50  0001 C CNN
 	1    1100 950
@@
 	1    0    0    -1
 $EndComp
-Text Label 8650 4100 0    50   ~ 0
+Text Label 9900 4100 0    50   ~ 0
 VOUT
 $Comp
@@
 $EndComp
 Wire Wire Line
-	9350 4400 9350 4550
+	9350 4100 9350 4550
 Wire Wire Line
 	6300 4200 6450 4200
@@
 VOUT
 Wire Wire Line
-	9150 4400 9150 4550
-Wire Wire Line
-	8950 4400 8950 4550
-Wire Wire Line
-	8750 4400 8750 4550
-Wire Wire Line
-	8550 4400 8550 4550
+	9150 4100 9150 4550
+Wire Wire Line
+	8950 4100 8950 4550
+Wire Wire Line
+	8750 4100 8750 4550
+Wire Wire Line
+	8550 4100 8550 4550
 Wire Wire Line
 	8550 4850 8550 5400
@@
 	8000 4100 8350 4100
 Wire Wire Line
-	8350 4550 8350 4400
+	8350 4550 8350 4100
+Wire Wire Line
+	9600 4100 9900 4100
+Wire Wire Line
+	8350 4100 8550 4100
 Connection ~ 8350 4100
-Wire Wire Line
-	8350 4100 8650 4100
-Wire Wire Line
-	8350 4400 8550 4400
-Connection ~ 8350 4400
-Wire Wire Line
-	8350 4400 8350 4100
-Connection ~ 8550 4400
-Wire Wire Line
-	8550 4400 8750 4400
-Connection ~ 8750 4400
-Wire Wire Line
-	8750 4400 8950 4400
-Connection ~ 8950 4400
-Wire Wire Line
-	8950 4400 9150 4400
-Connection ~ 9150 4400
-Wire Wire Line
-	9150 4400 9350 4400
+Connection ~ 8550 4100
+Wire Wire Line
+	8550 4100 8750 4100
+Connection ~ 8750 4100
+Wire Wire Line
+	8750 4100 8950 4100
+Connection ~ 8950 4100
+Wire Wire Line
+	8950 4100 9150 4100
+Connection ~ 9150 4100
+Wire Wire Line
+	9150 4100 9350 4100
 Wire Wire Line
 	6300 4400 7550 4400
@@
 NoConn ~ 6300 4300
 $Comp
-L AREA_composant:SIC461ED-T1-GE3 U1
+L Carte_Alim_V5-rescue:SIC461ED-T1-GE3-AREA_composant U1
 U 1 1 61E2315C
 P 5400 4600
@@
 Wire Wire Line
 	2650 4600 2900 4600
+$Comp
+L Device:R R10
+U 1 1 61E33A35
+P 9600 4700
+F 0 "R10" H 9670 4746 50  0000 L CNN
+F 1 "10k" H 9670 4655 50  0000 L CNN
+F 2 "Resistor_SMD:R_0603_1608Metric_Pad0.98x0.95mm_HandSolder" V 9530 4700 50  0001 C CNN
+F 3 "~" H 9600 4700 50  0001 C CNN
+	1    9600 4700
+	1    0    0    -1
+$EndComp
+Wire Wire Line
+	9600 4550 9600 4100
+$Comp
+L Device:LED D2
+U 1 1 61E33A3C
+P 9600 5150
+F 0 "D2" V 9639 5032 50  0000 R CNN
+F 1 "LED" V 9548 5032 50  0000 R CNN
+F 2 "LED_SMD:LED_0805_2012Metric_Pad1.15x1.40mm_HandSolder" H 9600 5150 50  0001 C CNN
+F 3 "~" H 9600 5150 50  0001 C CNN
+	1    9600 5150
+	0    -1   -1   0
+$EndComp
+Wire Wire Line
+	9600 4850 9600 5000
+Wire Wire Line
+	9600 5300 9600 5400
+Wire Wire Line
+	9350 4100 9600 4100
+Connection ~ 9350 4100
+Connection ~ 9600 4100
+Wire Wire Line
+	9600 5400 9350 5400
+Connection ~ 9350 5400
 $EndSCHEMATC
