File: Carte_Alim_V5/Carte_Alim_V5.kicad_pcb (KiCad board)
At the start: 2 copper layers, 71 parts, among them J1 BAT_IN, J10 12VC, J11 12VC, J12 12VC, J13 12VP, J14 12VP, J15 12VP, J16 12VP, J17 12VP, J18 12VP, J19 5VC, J2 BAT_IN, J20 5V_CAN, J21 5VC, J22 5V_CAN, J23 5VC, J24 5V_CAN, J25 5VC, J26 5V_CAN, J27 5VP, J28 5VP, J29 5VP, J3 MOT_OUT, J30 5VP, J31 5VP, J32 5VP, J4 MOT_OUT, J5 MOT_OUT, J6 MOT_OUT, J7 12VC, J8 12VC, J9 12VC, U1 LM2678S-5.0, U2 LM2678S-12, U3 LM2678S-12

Commit message: finalizing routing for test pcb buck
Parts:
- removed C20: 10n, Capacitor_SMD:C_0805_2012Metric_Pad1.18x1.45mm_HandSolder
- removed C21: 330u, Capacitor_SMD:CP_Elec_8x6.2
- removed C22: 100n, Capacitor_SMD:C_0805_2012Metric_Pad1.18x1.45mm_HandSolder
- removed D2, D3: S8KC-13, Diode_SMD:D_SMC_Handsoldering
- removed F1: 3557-2, AREA_lib_composant:FUSE_3557-2
- removed J10, J11, J12, J7, J8, J9: 12VC, AREA_lib_Connector:Wuerth_2.54mm_2pins_61900211121
- removed J13, J14, J15, J16, J17, J18: 12VP, AREA_lib_Connector:Wuerth_3.96mm_2pin_645002114822
- removed J19, J21, J23, J25: 5VC, AREA_lib_Connector:Wuerth_2.54mm_2pins_61900211121
- removed J20, J22, J24, J26: 5V_CAN, AREA_lib_Connector:690367290476
- removed J27, J28, J29, J30, J31, J32: 5VP, AREA_lib_Connector:Wuerth_3.96mm_2pin_645002114822
- removed J3, J4, J5, J6: MOT_OUT, AREA_lib_Connector:Wuerth_batcon_691313710002
- removed L2, L3: MSS1210-153MED, Inductor_SMD:L_12x12mm_H8mm
- removed PS1, PS2, PS3: TSR_2-2450, AREA_lib_composant:CONV_TSR_2-2450
- removed U2, U3: LM2678S-12, AREA_lib_composant:TO127P1435X464-8N
- added R1: 10k, Resistor_SMD:R_0603_1608Metric_Pad1.05x0.95mm_HandSolder, F.Cu at (61.2, 40.8)
- added R2: 2k, Resistor_SMD:R_0603_1608Metric_Pad1.05x0.95mm_HandSolder, F.Cu at (97.2, 42.2)
- added R3: 562k, Resistor_SMD:R_0603_1608Metric_Pad1.05x0.95mm_HandSolder, F.Cu at (92.0, 38.9)
- added R4: 226k, Resistor_SMD:R_0603_1608Metric_Pad1.05x0.95mm_HandSolder, F.Cu at (93.5, 38.9)
- added R5: 88.7k, Resistor_SMD:R_0603_1608Metric_Pad1.05x0.95mm_HandSolder, F.Cu at (97.8, 47.0)
- added R6: 100k, Resistor_SMD:R_0603_1608Metric_Pad1.05x0.95mm_HandSolder, F.Cu at (97.5, 44.8)
- added R7: 3.3, Resistor_SMD:R_0603_1608Metric_Pad1.05x0.95mm_HandSolder, F.Cu at (90.2, 39.0)
- added R8: 52.3k, Resistor_SMD:R_0603_1608Metric_Pad1.05x0.95mm_HandSolder, F.Cu at (105.2, 50.0)
- added R9: 10k, Resistor_SMD:R_0603_1608Metric_Pad1.05x0.95mm_HandSolder, F.Cu at (103.5, 50.0)
- C1: value 82u -> 100n; footprint Capacitor_SMD:CP_Elec_8x6.9 -> Capacitor_SMD:C_0805_2012Metric_Pad1.15x1.40mm_HandSolder
- C10, C11: value 10u -> 1u; footprint Capacitor_THT:CP_Radial_D4.0mm_P2.00mm -> Capacitor_SMD:C_0805_2012Metric_Pad1.15x1.40mm_HandSolder
- C12: value 47u -> 100n; footprint Capacitor_THT:CP_Radial_D4.0mm_P2.00mm -> Capacitor_SMD:C_0805_2012Metric_Pad1.15x1.40mm_HandSolder
- C13: value 10u -> 22u; footprint Capacitor_THT:CP_Radial_D4.0mm_P2.00mm -> Capacitor_SMD:C_1210_3225Metric_Pad1.42x2.65mm_HandSolder
- C14, C15: value 47u -> 22u; footprint Capacitor_THT:CP_Radial_D4.0mm_P2.00mm -> Capacitor_SMD:C_1210_3225Metric_Pad1.42x2.65mm_HandSolder
- C16, C17, C4, C5: value 100n -> 22u; footprint Capacitor_SMD:C_0805_2012Metric_Pad1.18x1.45mm_HandSolder -> Capacitor_SMD:C_1210_3225Metric_Pad1.42x2.65mm_HandSolder
- C18, C3: value 330u -> 22u; footprint Capacitor_SMD:CP_Elec_10x12.6 -> Capacitor_SMD:C_1210_3225Metric_Pad1.42x2.65mm_HandSolder
- C19: footprint Capacitor_SMD:C_0805_2012Metric_Pad1.18x1.45mm_HandSolder -> Capacitor_SMD:C_0805_2012Metric_Pad1.15x1.40mm_HandSolder
- C2: value 82u -> 22u; footprint Capacitor_SMD:CP_Elec_8x6.9 -> Capacitor_SMD:C_1210_3225Metric_Pad1.42x2.65mm_HandSolder
- C6, C7: value 10n -> 22u; footprint Capacitor_SMD:C_0805_2012Metric_Pad1.18x1.45mm_HandSolder -> Capacitor_SMD:C_1210_3225Metric_Pad1.42x2.65mm_HandSolder
- C8: value 330u -> 33n; footprint Capacitor_SMD:CP_Elec_8x6.2 -> Capacitor_SMD:C_0805_2012Metric_Pad1.15x1.40mm_HandSolder
- C9: value 330u -> 100n; footprint Capacitor_SMD:CP_Elec_8x6.2 -> Capacitor_SMD:C_0805_2012Metric_Pad1.15x1.40mm_HandSolder
- D1: value S8KC-13 -> LED; footprint Diode_SMD:D_SMC_Handsoldering -> LED_SMD:LED_0805_2012Metric_Pad1.15x1.40mm_HandSolder
- L1: value MSS1210-153MED -> 4.7uH; footprint Inductor_SMD:L_12x12mm_H8mm -> Inductor_SMD:L_Vishay_IHLP-6767
- U1: value LM2678S-5.0 -> SIC466ED-T1-GE3; footprint AREA_lib_composant:TO127P1435X464-8N -> AREA_lib_composant:CONV_SIC461ED-T1-GE3
- moved H1 184.1 mm to (42.4, 33.0)
- moved H4 182.8 mm to (42.2, 74.8)
- moved H3 128.2 mm to (145.2, 32.9)
- moved C10 113.2 mm to (95.0, 52.5), turned to 180 degrees
- moved H2 109.4 mm to (145.2, 74.8)
- moved C12 106.2 mm to (110.0, 50.0), turned to 90 degrees
- moved C15 104.0 mm to (127.8, 50.0), turned to 90 degrees
- moved D1 93.5 mm to (65.0, 40.8)
- moved C13 93.3 mm to (131.5, 50.0), turned to 90 degrees
- moved J2 88.2 mm to (137.4, 48.2), turned to 90 degrees
- moved C6 82.8 mm to (81.9, 47.0)
- moved C2 78.7 mm to (68.5, 47.0), turned to 270 degrees
- moved C11 76.1 mm to (101.0, 44.8), turned to 180 degrees
- moved C4 74.6 mm to (85.2, 47.0), turned to 270 degrees
- moved L1 67.3 mm to (95.6, 63.5), turned to 0 degrees
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Connections:
- C1 pad 1: +24V -> +BATT
- C10 pad 1: +24V -> GND
- C10 pad 2: GND -> Net-(C10-Pad2)
- C11 pad 1: +24V -> GND
- C11 pad 2: GND -> /VDD
- C12 pad 1: +5V -> /VOUT
- C13 pad 1: +24V -> /VOUT
- C14 pad 1: +12C -> /VOUT
- C15 pad 1: +5C -> /VOUT
- C16 pad 1: +5P -> /VOUT
- C17 pad 1: +12P -> /VOUT
- C18 pad 1: +24V -> /VOUT
- C19 pad 1: +24V -> +BATT
- C2 pad 1: +24V -> +BATT
- C3 pad 1: +24V -> +BATT
- C4 pad 1: +24V -> +BATT
- C5 pad 1: +24V -> +BATT
- C6 pad 1: Net-(C6-Pad1) -> +BATT
- C6 pad 2: Net-(C6-Pad2) -> GND
- C7 pad 1: Net-(C7-Pad1) -> +BATT
- C7 pad 2: Net-(C7-Pad2) -> GND
- C8 pad 1: +5P -> Net-(C8-Pad1)
- C9 pad 1: +12P -> Net-(C9-Pad1)
- C9 pad 2: GND -> Net-(C9-Pad2)
- D1 pad 1: Net-(C6-Pad2) -> GND
- D1 pad 2: GND -> Net-(D1-Pad2)
- J2 pad 1: +BATT -> /VOUT
- L1 pad 1: Net-(C6-Pad2) -> Net-(L1-Pad1)
- L1 pad 2: +5P -> /VOUT
- U1 pad 1: Net-(C6-Pad2) -> +BATT
- U1 pad 2: +24V -> Net-(R6-Pad2)
- U1 pad 3: Net-(C6-Pad1) -> Net-(R3-Pad2)
- U1 pad 4: GND -> Net-(R7-Pad1)
- U1 pad 5: Net-(U1-Pad5) -> Net-(C9-Pad2)
- U1 pad 6: +5P -> Net-(C9-Pad2)
- U1 pad 7: Net-(U1-Pad7) -> +BATT
- U1 pad 8: GND -> +BATT
Routing:
- net Net-(C6-Pad2): track 11.5 -> 0.00 mm
- net GND: track 0.00 -> 6.55 mm
- added copper zone on F.Cu, net +BATT
- added copper zone on F.Cu, net /VOUT
- added copper zone on B.Cu, net GND
- added copper zone on F.Cu, net Net-(L1-Pad1)
- removed copper zone on F.Cu, net +24V
- removed copper zone on F.Cu, net +5P
- removed copper zone on F.Cu, net Net-(C6-Pad2)

Commit message: last version of alim v5
Parts:
- added D2: LED, LED_SMD:LED_0805_2012Metric_Pad1.15x1.40mm_HandSolder, F.Cu at (124.0, 41.5)
- added R10: 10k, Resistor_SMD:R_0603_1608Metric_Pad0.98x0.95mm_HandSolder, F.Cu at (124.2, 43.2)
- J1, J2: footprint AREA_lib_Connector:Wuerth_batcon_691313710002 -> Connector_Phoenix_MSTB:PhoenixContact_MSTBVA_2,5_2-G-5,08_1x02_P5.08mm_Vertical
- moved H4 26.4 mm to (68.2, 70.2)
- moved H1 26.2 mm to (68.2, 37.2)
- moved C13 19.0 mm to (113.2, 55.2), turned to 270 degrees
- moved D1 17.1 mm to (69.5, 57.2)
- moved H2 17.1 mm to (128.8, 70.2)
- moved H3 17.1 mm to (128.8, 37.2)
- moved R1 17.0 mm to (69.6, 55.5), turned to 180 degrees
- moved C2 14.7 mm to (82.5, 42.5), turned to 90 degrees
- moved C15 12.1 mm to (117.0, 55.2), turned to 270 degrees
- moved J2 10.7 mm to (128.0, 53.2)
- moved C3 8.45 mm to (79.0, 42.5), turned to 90 degrees
- moved J1 8.31 mm to (68.5, 45.2)
- moved C16 6.28 mm to (120.7, 55.2), turned to 270 degrees
- moved C5 4.51 mm to (75.5, 42.5), turned to 90 degrees
- moved R6 4.07 mm to (94.8, 41.8), turned to 270 degrees
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Connections:
- U1 pad 15: Net-(U1-Pad15) -> (no net)
- U1 pad 18: Net-(U1-Pad18) -> (no net)
- U1 pad 21: Net-(U1-Pad21) -> (no net)
Routing:
- net +BATT: track 0.00 -> 30.1 mm, vias 0 -> 2
- net /VOUT: track 0.00 -> 27.1 mm, vias 0 -> 1
- net /VDD: track 0.00 -> 15.3 mm
- net Net-(R8-Pad1): track 0.00 -> 12.3 mm
- net Net-(R2-Pad1): track 0.00 -> 4.78 mm
- net Net-(C8-Pad1): track 0.00 -> 4.08 mm
- net Net-(C9-Pad2): track 0.00 -> 4.03 mm
- net Net-(R3-Pad2): track 0.00 -> 3.74 mm
- net Net-(R7-Pad1): track 0.00 -> 3.66 mm
- net Net-(R6-Pad2): track 0.00 -> 2.60 mm
- net Net-(R5-Pad1): track 0.00 -> 2.10 mm
- net Net-(D1-Pad2): track 0.00 -> 1.86 mm
- net Net-(C9-Pad1): track 0.00 -> 1.79 mm
- net Net-(C10-Pad2): track 0.00 -> 1.74 mm
- net Net-(D2-Pad2): track 0.00 -> 1.61 mm
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Other:
- board outline added: 68 x 40.5 mm
- board text added: "Buck Proto v1 SIC466"
- board text added: "VIN"
- board text added: "VOUT"
- board text added: "Vin = 4.5-60V"

Commit message: lots of stuf
Other:
- net class Default removed
