File: PCB_AX12/PCB_AX12.kicad_sch (KiCad schematic)
At the start: 48 parts, among them J1 12VP, J2 CON_CAN, J3 USB_C_Receptacle_USB2.0, J4 CON_CAN, J5 ax12, J6 ax12, J7 ax12, J8 ax12, SW1 BOOT, SW2 RST, U1 SN65HVD232, U2 NCP1117-3.3_SOT223, U3 STM32F302C6Tx, Y1 8MHz

Commit message: PCB RMEAS ok to fab
Parts:
- D3: value LED_5V -> LED_12V
- D4: value LED_DEBUG -> LED_5V
- R5: value 560 -> 1k
- R8: value 270 -> 1k
- gave numbers to parts that had none: 2
Connections:
- net +5V: now also D4.2 (A)
- net at U3.37 (PA14): no longer D4.2 (A)
