File: PCB_AX12/PCB_AX12.kicad_pcb (KiCad board)
At the start: 2 copper layers, 62 x 45.2 mm, 48 parts, among them J1 12VP, J2 CON_CAN, J3 USB_C_Receptacle_USB2.0, J4 CON_CAN, J5 ax12, J6 ax12, J7 ax12, J8 ax12, U1 SN65HVD232, U2 NCP1117-3.3_SOT223, U3 STM32F302C6Tx, Y1 8MHz

Commit message: Beaucoup de chose
Routing:
- net GND: track 11.6 -> 17.2 mm
Changed lines of the file:
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@@
     (property "Sheetfile" "PCB_AX12.kicad_sch")
     (property "Sheetname" "")
+    (zone_connect 1)
     (attr through_hole)
     (fp_text reference "J3" (at 2.975 1.8 unlocked) (layer "B.SilkS")
@@
   (segment (start 126.25 108.75) (end 128.75 108.75) (width 0.4) (layer "F.Cu") (net 1))
   (segment (start 121.4625 111.25) (end 122.5 110.2125) (width 0.4) (layer "F.Cu") (net 1))
+  (segment (start 117.5 108) (end 116.38 108) (width 0.127) (layer "F.Cu") (net 2))
+  (segment (start 123.475 107.925) (end 123.475 108.575) (width 0.127) (layer "F.Cu") (net 2))
   (segment (start 121.75 96.6625) (end 121.75 98.05) (width 0.25) (layer "F.Cu") (net 2))
   (segment (start 118.75 88.3375) (end 118.75 86.75) (width 0.25) (layer "F.Cu") (net 2))
   (segment (start 133.925 87.9) (end 133.75 88.075) (width 0.4) (layer "F.Cu") (net 2))
   (segment (start 115.3375 94.75) (end 113.6 94.75) (width 0.25) (layer "F.Cu") (net 2))
+  (segment (start 123.5 107.95) (end 124.57 107.95) (width 0.127) (layer "F.Cu") (net 2))
+  (segment (start 123.475 107.225) (end 123.475 107.925) (width 0.127) (layer "F.Cu") (net 2))
   (segment (start 123.6625 90.25) (end 124.75 90.25) (width 0.25) (layer "F.Cu") (net 2))
   (segment (start 130.635 88.6525) (end 131.0375 88.25) (width 0.4) (layer "F.Cu") (net 2))
   (segment (start 130.635 90.775) (end 130.635 88.6525) (width 0.4) (layer "F.Cu") (net 2))
+  (segment (start 123.475 107.925) (end 123.5 107.95) (width 0.127) (layer "F.Cu") (net 2))
   (segment (start 124.75 90.25) (end 125.15 89.85) (width 0.25) (layer "F.Cu") (net 2))
+  (segment (start 124.57 107.95) (end 124.825 108.205) (width 0.127) (layer "F.Cu") (net 2))
+  (segment (start 117.525 107.225) (end 117.525 107.975) (width 0.127) (layer "F.Cu") (net 2))
+  (segment (start 117.525 107.975) (end 117.5 108) (width 0.127) (layer "F.Cu") (net 2))
+  (segment (start 117.525 107.975) (end 117.525 108.575) (width 0.127) (layer "F.Cu") (net 2))
+  (segment (start 116.38 108) (end 116.175 108.205) (width 0.127) (layer "F.Cu") (net 2))
   (segment (start 136.2 87.9) (end 133.925 87.9) (width 0.4) (layer "F.Cu") (net 2))
   (via (at 121.7 86.7) (size 0.6) (drill 0.3) (layers "F.Cu" "B.Cu") (free) (net 2))
