File: PCB_BAT/PCB_BAT.kicad_pcb (KiCad board)
At the start: 2 copper layers, 62.2 x 25.8 mm, 7 parts, among them J1 BATT, J2 BATT, J3 BATT, J4 BATT, K1 SANYOU_SRD_Form_C

Commit message: Beaucoup de chose
Parts:
- moved D1 15.3 mm to (102.2, 75.4), turned to 90 degrees
- renumbered BAU to SW1
Connections:
- D1 pad 1: GND -> Net-(K1-Pad2)
- D1 pad 2: Net-(D1-Pad2) -> GND
- K1 pad 2: Net-(D1-Pad2) -> Net-(K1-Pad2)
- SW1 pad 2: Net-(D1-Pad2) -> Net-(K1-Pad2)
Routing:
- net Net-(K1-Pad2): track 0.00 -> 13.1 mm
- net Net-(D1-Pad2): track 13.1 -> 0.00 mm
Changed lines of the file:
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@@
   (net 0 "")
   (net 1 "GND")
-  (net 2 "Net-(D1-Pad2)")
+  (net 2 "Net-(K1-Pad2)")
   (net 3 "+BATT")
   (net 4 "/OUT")
@@
   (net 6 "unconnected-(SW1-Pad3)")
   (footprint "Diode_THT:D_DO-201AD_P15.24mm_Horizontal" (layer "F.Cu")
-    (at 102.25 60.13 -90)
+    (at 102.2 75.4 90)
     (descr "Diode, DO-201AD series, Axial, Horizontal, pin pitch=15.24mm, , length*diameter=9.5*5.2mm^2, , http://www.diodes.com/_files/packages/DO-201AD.pdf")
     (tags "Diode DO-201AD series Axial Horizontal pin pitch 15.24mm  length 9.5mm diameter 5.2mm")
@@
     (fp_line (start 12.37 2.6) (end 12.37 -2.6) (layer "F.Fab") (width 0.1))
     (fp_line (start 2.87 -2.6) (end 2.87 2.6) (layer "F.Fab") (width 0.1))
-    (pad "1" thru_hole rect (at 0 0 270) (size 3.2 3.2) (drill 1.6) (layers *.Cu *.Mask)
-      (net 1 "GND") (pinfunction "K") (pintype "input"))
-    (pad "2" thru_hole oval (at 15.24 0 270) (size 3.2 3.2) (drill 1.6) (layers *.Cu *.Mask)
-      (net 2 "Net-(D1-Pad2)") (pinfunction "A") (pintype "input"))
+    (pad "1" thru_hole rect (at 0 0 90) (size 3.2 3.2) (drill 1.6) (layers *.Cu *.Mask)
+      (net 2 "Net-(K1-Pad2)") (pinfunction "K") (pintype "passive"))
+    (pad "2" thru_hole oval (at 15.24 0 90) (size 3.2 3.2) (drill 1.6) (layers *.Cu *.Mask)
+      (net 1 "GND") (pinfunction "A") (pintype "passive"))
     (model "${KICAD6_3DMODEL_DIR}/Diode_THT.3dshapes/D_DO-201AD_P15.24mm_Horizontal.wrl"
       (offset (xyz 0 0 0))
@@
     (property "Sheetname" "")
     (attr through_hole)
-    (fp_text reference "BAU" (at 0 -7.46) (layer "F.SilkS")
+    (fp_text reference "SW1" (at 0 -7.46) (layer "F.SilkS")
       (effects (font (size 1 1) (thickness 0.15)))
     )
@@
       (net 3 "+BATT") (pinfunction "A") (pintype "passive"))
     (pad "2" thru_hole oval (at 0 2.54) (size 1.7 1.7) (drill 1) (layers *.Cu *.Mask)
-      (net 2 "Net-(D1-Pad2)") (pinfunction "B") (pintype "passive"))
+      (net 2 "Net-(K1-Pad2)") (pinfunction "B") (pintype "passive"))
     (pad "3" thru_hole oval (at 0 5.08) (size 1.7 1.7) (drill 1) (layers *.Cu *.Mask)
       (net 6 "unconnected-(SW1-Pad3)") (pinfunction "C") (pintype "passive+no_connect"))
@@
       (net 3 "+BATT") (pintype "passive"))
     (pad "2" thru_hole circle (at 1.95 6.05 90) (size 2.5 2.5) (drill 1) (layers *.Cu *.Mask)
-      (net 2 "Net-(D1-Pad2)") (pintype "passive"))
+      (net 2 "Net-(K1-Pad2)") (pintype "passive"))
     (pad "3" thru_hole circle (at 14.15 6.05 90) (size 3 3) (drill 1.3) (layers *.Cu *.Mask)
       (net 5 "unconnected-(K1-Pad3)") (pintype "passive+no_connect"))
@@
   )
   (segment (start 102.25 75.37) (end 108.38 75.37) (width 1.5) (layer "F.Cu") (net 2))
+  (segment (start 102.12 75.5) (end 102.25 75.37) (width 1.5) (layer "F.Cu") (net 2))
+  (segment (start 108.38 75.37) (end 109.7 74.05) (width 1.5) (layer "F.Cu") (net 2))
   (segment (start 97.25 75.5) (end 102.12 75.5) (width 1.5) (layer "F.Cu") (net 2))
-  (segment (start 108.38 75.37) (end 109.7 74.05) (width 1.5) (layer "F.Cu") (net 2))
-  (segment (start 102.12 75.5) (end 102.25 75.37) (width 1.5) (layer "F.Cu") (net 2))
   (zone (net 3) (net_name "+BATT") (layers F&B.Cu) (hatch edge 0.508)
     (priority 1)
@@
     (polygon
       (pts
+        (xy 133 67.3)
+        (xy 127.2 67.3)
+        (xy 127.2 74.5)
+        (xy 133 74.502261)
         (xy 133 79.75)
-        (xy 127 79.75)
-        (xy 127 66.25)
+        (xy 119 79.75)
+        (xy 119 66.25)
         (xy 119 66.25)
         (xy 119 59.25)
