File: PCB_BAT/PCB_BAT.kicad_sch (KiCad schematic)
At the start: 7 parts, among them J1 BATT, J2 BATT, J3 BATT, J4 BATT, K1 SANYOU_SRD_Form_C, SW1 BAU

Commit message: Beaucoup de chose
Parts:
- D1: symbol pspice:DIODE -> Diode:1N5408
Connections:
- net GND: now also D1.2 (A); no longer D1.1 (K)
- net at K1.2, SW1.2 (B): now also D1.1 (K); no longer D1.2 (A)
Changed lines of the file:
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@@
     (stroke (width 0) (type default) (color 0 0 0 0))
   )
-  (wire (pts (xy 107.95 33.02) (xy 119.38 33.02))
+  (wire (pts (xy 106.68 33.02) (xy 119.38 33.02))
     (stroke (width 0) (type default) (color 0 0 0 0))
   )
@@
     (stroke (width 0) (type default) (color 0 0 0 0))
   )
-  (wire (pts (xy 97.79 33.02) (xy 92.71 33.02))
+  (wire (pts (xy 92.71 33.02) (xy 99.06 33.02))
     (stroke (width 0) (type default) (color 0 0 0 0))
   )
@@
     (pin "1")
   )
-  (symbol (lib_id "pspice:DIODE") (at 102.87 33.02 180) (unit 1)
+  (symbol (lib_id "Diode:1N5408") (at 102.87 33.02 0) (unit 1)
     (in_bom yes) (on_board yes) (fields_autoplaced)
-    (property "Reference" "D1" (id 0) (at 102.87 26.9072 0))
-    (property "Value" "1N5408" (id 1) (at 102.87 29.4441 0))
-    (property "Footprint" "Diode_THT:D_DO-201AD_P15.24mm_Horizontal" (id 2) (at 102.87 33.02 0)
+    (property "Reference" "D1" (id 0) (at 102.87 28.0502 0))
+    (property "Value" "1N5408" (id 1) (at 102.87 30.5871 0))
+    (property "Footprint" "Diode_THT:D_DO-201AD_P15.24mm_Horizontal" (id 2) (at 102.87 37.465 0)
       (effects (font (size 1.27 1.27)) hide)
     )
-    (property "Datasheet" "~" (id 3) (at 102.87 33.02 0)
+    (property "Datasheet" "http://www.vishay.com/docs/88516/1n5400.pdf" (id 3) (at 102.87 33.02 0)
       (effects (font (size 1.27 1.27)) hide)
     )
