File: PCB_dev_stm32f302/PCB_dev_stm32f302.kicad_pcb (KiCad board)
At the start: 2 copper layers, 51 x 18.5 mm, 32 parts, among them J1 USB_C_Receptacle_USB2.0, J2 HEADER_PA, J3 Conn_01x05_Male, J4 HEADER_PB, SW1 BOOT, SW2 RST, U1 STM32F302C6Tx, U2 NCP1117-3.3_SOT223, Y1 8MHz

Commit message: Beaucoup de chose
Parts:
- removed J3: Conn_01x05_Male, Connector_PinHeader_2.54mm:PinHeader_1x05_P2.54mm_Vertical
- moved C9 0.90 mm to (126.5, 109.6)
- moved C4 0.42 mm to (121.8, 100.8)
- moved R2 0.42 mm to (118.3, 100.8)
- moved C1 0.34 mm to (125.2, 100.8)
- moved C12 0.30 mm to (128.8, 100.8)
- moved C2 0.15 mm to (126.5, 108.1)
- moved U1 0.15 mm to (134.3, 105.0)
Connections:
- J1 pad A8: (no net) -> unconnected-(J1-PadA8)
- J1 pad B8: (no net) -> unconnected-(J1-PadB8)
- J2 pad 15: /PA15 -> GND
- J4 pad 1: /PB3 -> +5V
- J4 pad 10: /PB13 -> /PB9
- J4 pad 11: /PB14 -> /PB15
- J4 pad 12: /PB15 -> /PB14
- J4 pad 13: GND -> /PB13
- J4 pad 14: +3V3 -> /PB11
- J4 pad 15: +5V -> /PB10
- J4 pad 2: /PB4 -> +3V3
- J4 pad 3: /PB5 -> GND
- J4 pad 4: /PB6 -> /PB3
- J4 pad 5: /PB7 -> /PB4
- J4 pad 6: /PB8 -> /PB5
- J4 pad 7: /PB9 -> /PB6
- J4 pad 8: /PB10 -> /PB7
- J4 pad 9: /PB11 -> /PB8
- U1 pad 1: (no net) -> unconnected-(U1-Pad1)
- U1 pad 2: (no net) -> unconnected-(U1-Pad2)
- U1 pad 3: (no net) -> unconnected-(U1-Pad3)
- U1 pad 37: (no net) -> /SWCLK
- U1 pad 4: (no net) -> unconnected-(U1-Pad4)
Routing:
- net +5V: track 82.4 -> 40.8 mm, vias 1 -> 2
- net +3V3: track 68.5 -> 34.8 mm, vias 1 -> 10
- net /BOOT0: track 2.37 -> 25.5 mm
- net /USB-: track 0.00 -> 19.0 mm
- net /USB+: track 0.00 -> 18.5 mm
- net /PA10: track 0.00 -> 18.0 mm
- net /PB10: track 6.06 -> 22.4 mm
- net /PA9: track 0.00 -> 14.3 mm
- net Net-(J1-PadA5): track 0.00 -> 13.0 mm, vias 0 -> 1
- net /PA8: track 0.00 -> 12.3 mm
- net /PB8: track 12.6 -> 3.08 mm
- net /PB7: track 15.6 -> 6.95 mm
- net Net-(C1-Pad1): track 0.00 -> 8.36 mm
- net /PB11: track 12.6 -> 20.6 mm
- net /PB9: track 10.9 -> 3.35 mm, vias 1 -> 0
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- added copper zone on In1.Cu, net +3V3
- added copper zone on B.Cu, net GND
- added copper zone on F.Cu, net GND
- added copper zone on In2.Cu, net GND
Other:
- board size 51 x 18.5 mm -> 51 x 19.7 mm
- copper layers 2 -> 4
- net class Default removed
- board text added: "3V3"
- board text added: "5V"
- board text added: "A0"
- board text added: "A1"
- board text added: "A10"
- board text added: "A2"
- board text added: "A3"
- board text added: "A4"
- board text added: "A5"
- board text added: "A6"
- board text added: "A7"
- board text added: "A8"
- board text added: "A9"
- board text added: "B0"
- board text added: "B1"
- board text added: "B10"
- board text added: "B11"
- board text added: "B13"
- board text added: "B14"
- board text added: "B15"
- board text added: "B2"
- board text added: "B3"
- board text added: "B4"
- board text added: "B5"
- board text added: "B6"
- board text added: "B7"
- board text added: "B8"
- board text added: "B9"
- board text added: "BOOT"
- board text added: "GND"
- board text added: "Nukleo STM32F302"
- board text added: "RESET"
