File: Carte_Alim_V6_2022/REGULO.kicad_sch (KiCad schematic)
At the start: 29 parts, among them U1 SIC466ED-T1-GE3

Commit message: modif carte alim
Parts:
- removed C5, C6: 22u, Capacitor_SMD:C_1210_3225Metric_Pad1.33x2.70mm_HandSolder, symbol Device:C
- renumbered C1 to C35, C2 to C36, C3 to C37, C4 to C38, C7 to C41, C8 to C42, C9 to C43, C10 to C44, C11 to C45, C12 to C46, C13 to C47, C14 to C48, C15 to C49, C16 to C50, C17 to C51, D2 to D6, L1 to L3, R2 to R22, R3 to R23, R4 to R24, R5 to R25, R6 to R26, R7 to R27, R8 to R28, R9 to R29, R10 to R30, U1 to U3
Other:
- moved on the sheet: C45
