File: Carte_Alim_V6_2022/Carte_Alim_V6_2022.kicad_pcb (KiCad board)
At the start: 4 copper layers, 98.3 x 111.5 mm, 114 parts, among them J1 BAT_IN, J10 12VC, J11 12VC, J12 12VC, J13 12VP, J14 12VP, J15 12VP, J16 12VP, J17 12VP, J18 12VP, J19 5VC, J2 BAT_IN, J20 5V_CAN, J21 5VC, J22 5V_CAN, J23 5VC, J24 5V_CAN, J25 5VC, J26 5V_CAN, J27 5VP, J28 5VP, J29 5VP, J3 MOT_OUT, J30 5VP, J31 5VP, J32 5VP, J4 MOT_OUT, J5 MOT_OUT, J6 MOT_OUT, J7 12VC, J8 12VC, J9 12VC, U1 SIC466ED-T1-GE3, U3 SIC466ED-T1-GE3

Commit message: modif carte alim
Parts:
- removed C39, C40: 22u, Capacitor_SMD:C_1210_3225Metric_Pad1.33x2.70mm_HandSolder
- removed C54: 10u, Capacitor_THT:CP_Radial_D4.0mm_P2.00mm
- removed C57: 47u, Capacitor_THT:CP_Radial_D4.0mm_P2.00mm
- removed PS3: TSR_2-2450, AREA_lib_composant:CONV_TSR_2-2450
- added C18: 10u, Capacitor_SMD:C_1210_3225Metric_Pad1.33x2.70mm_HandSolder, F.Cu at (105.4, 65.3)
- added C19: 10u, Capacitor_SMD:C_1210_3225Metric_Pad1.33x2.70mm_HandSolder, F.Cu at (108.7, 65.3)
- added C20: 10n, Capacitor_SMD:C_0805_2012Metric_Pad1.18x1.45mm_HandSolder, F.Cu at (124.2, 65.2)
- added C21: 330u, Capacitor_SMD:CP_Elec_8x11.9, F.Cu at (134.5, 59.6)
- added C22: 100n, Capacitor_SMD:C_0805_2012Metric_Pad1.18x1.45mm_HandSolder, F.Cu at (140.9, 55.1)
- added C23: 10n, Capacitor_SMD:C_0805_2012Metric_Pad1.18x1.45mm_HandSolder, F.Cu at (140.9, 57.2)
- added D8: SSC54-E3/9AT, Diode_SMD:D_SOD-128, F.Cu at (129.5, 65.8)
- added D9: LED, LED_SMD:LED_0805_2012Metric_Pad1.15x1.40mm_HandSolder, F.Cu at (206.4, 29.0)
- added L2: 10uH, Inductor_SMD:L_Wuerth_HCM-7050, F.Cu at (126.2, 60.0)
- added R15: 10k, Resistor_SMD:R_0603_1608Metric_Pad0.98x0.95mm_HandSolder, F.Cu at (120.1, 58.8)
- added R16: 3k16, Resistor_SMD:R_0603_1608Metric_Pad0.98x0.95mm_HandSolder, F.Cu at (116.8, 58.8)
- added R17: 10k, Resistor_SMD:R_0603_1608Metric_Pad0.98x0.95mm_HandSolder, F.Cu at (202.8, 29.0)
- added U2: TPS5450ddar, Package_SO:TI_SO-PowerPAD-8_ThermalVias, F.Cu at (118.4, 63.4)
- C5, C6: value 22u -> 100n; footprint Capacitor_SMD:C_1210_3225Metric_Pad1.33x2.70mm_HandSolder -> Capacitor_SMD:C_0805_2012Metric_Pad1.18x1.45mm_HandSolder
- moved C5 34.1 mm to (111.4, 64.7)
- moved C6 32.5 mm to (113.5, 64.7), turned to -90 degrees
- moved C56 4.18 mm to (115.1, 55.4)
- moved C38 3.30 mm to (78.6, 98.8)
- moved C4 3.30 mm to (81.0, 64.5)
- moved C53 1.96 mm to (108.3, 55.3)
- moved C47 0.35 mm to (103.0, 111.5)
- moved C49 0.35 mm to (106.3, 111.5)
- moved C50 0.35 mm to (109.6, 111.5)
Connections:
- U1 pad A12: Net-(L1-Pad1) -> (no net)
- U3 pad A12: Net-(L3-Pad1) -> (no net)
Routing:
- net +5V: track 64.3 -> 23.4 mm
- net +24V: track 46.7 -> 39.8 mm, vias 19 -> 2
- net /REGULO5v/VSENS: track 0.00 -> 4.92 mm
- net GND: track 11.6 -> 16.5 mm, vias 187 -> 143
- net Net-(C20-Pad2): track 0.00 -> 2.09 mm
- net Net-(L3-Pad1): vias 22 -> 8
- net Net-(L1-Pad1): vias 23 -> 8
- net +12P: vias 17 -> 9
- added copper zone on B.Cu, net +5V
- added copper zone on F.Cu, net +5V
- added copper zone on F.Cu, net Net-(C20-Pad1)
