File: _Principal_V3/_Principal_V3.kicad_sch (KiCad schematic)
At the start: 57 parts, among them J1 CAN, J10 UART, J11 I2C, J12 NEXTION, J2 ENCODEUR_G, J3 ENCODEUR_D, J4 CAN, J5 MOTOR_D, J6 BATT, J7 MOTOR_G, J8 FAN, J9 FAN, U1 4504, U2 SN65HVD232, U3 DEV-14058

Commit message: Maj carte alim
Parts:
- U3: value DEV-14058 -> TEENSY 3.6
Connections:
- net sheet6220E40C/IN is gone; now on net Level_shifter/IN: R11.1
- net Level_shifter/IN: no longer J12.2 (Pin_2)
- net sheet6215AC10/IN renamed Level_shifter/IN
- net sheet6216318E/IN renamed Level_shifter/IN
- net sheet6216B4BD/IN renamed Level_shifter/IN
- net sheet6220E40B/IN renamed Level_shifter/IN
- new net Level_shifter/IN: J12.2 (Pin_2)
Other:
- removed sheet sheet6215AC10
- removed sheet sheet6216318E
- removed sheet sheet6216B4BD
- removed sheet sheet6220E40B
- removed sheet sheet6220E40C
- note added: "Encodeurs - AMT102"
- note added: "I²C"
- note added: "Nextion"
- note added: "UART"
- note added: "Ventilo"
- note removed: "Encodeurs - AMT103"
- moved on the sheet: C10, C11, C8, H1, H2, H3, H4, J10, J11, J12, J8, J9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
