File: PCB_Principal_V4/PCB_Principal_V4.kicad_pcb (KiCad board)
At the start: 2 copper layers, 82.8 x 56 mm, 54 parts, among them J1 CAN, J10 NEXTION, J2 ENCODEUR_G, J3 ENCODEUR_D, J4 FAN, J5 CAN, J6 MOTOR_D, J7 BATT, J8 FAN, J9 MOTOR_G, Q1 Q_NPN_BEC, Q2 Q_NPN_BEC, Q3 SI2302S, Q4 SI2302S, U1 4504, U2 SN65HVD232, U3 TEENSY 4.1

Commit message: update last PCBs
Parts:
- added D7: 1N4148W, Diode_SMD:D_SOD-123, F.Cu at (166.9, 94.1)
- added D8: 1N4148W, Diode_SMD:D_SOD-123, F.Cu at (166.9, 88.3)
- added J11: FAN, AREA_lib_Connector:Wuerth_2.54mm_2pins_61900211121, F.Cu at (171.4, 93.7)
- added J12: FAN, AREA_lib_Connector:Wuerth_2.54mm_2pins_61900211121, F.Cu at (171.4, 87.8)
- added Q5: Q_NPN_BEC, Package_TO_SOT_SMD:SOT-23, F.Cu at (164.0, 94.6)
- added Q6: Q_NPN_BEC, Package_TO_SOT_SMD:SOT-23, F.Cu at (164.0, 88.7)
- added R11: 10k, Resistor_SMD:R_0805_2012Metric_Pad1.20x1.40mm_HandSolder, F.Cu at (163.8, 91.6)
- added R12: 10k, Resistor_SMD:R_0805_2012Metric_Pad1.20x1.40mm_HandSolder, F.Cu at (163.8, 85.7)
- moved D2 8.83 mm to (164.1, 82.6)
- moved D3 8.83 mm to (166.2, 82.6)
- moved D4 8.83 mm to (168.6, 82.6)
- moved R3 8.83 mm to (164.1, 78.8)
- moved R4 8.83 mm to (166.2, 78.8)
- moved R5 8.83 mm to (168.6, 78.8)
- moved R1 0.12 mm to (160.7, 100.6)
Connections:
- U3 pad 29: unconnected-(U3-Pad29) -> /PWM_FAN4
- U3 pad 30: unconnected-(U3-Pad30) -> /PWM_FAN3
Routing:
- net +24V: track 61.3 -> 82.9 mm, vias 1 -> 0
- net /PWM_FAN4: track 0.00 -> 18.4 mm
- net /CANH: track 39.3 -> 51.1 mm
- net /CANL: track 32.8 -> 44.2 mm, vias 2 -> 0
- net /PWM_FAN3: track 0.00 -> 10.8 mm
- net Net-(D7-Pad2): track 0.00 -> 7.58 mm
- net Net-(D8-Pad2): track 0.00 -> 7.56 mm
- net +5V: track 223.7 -> 231.2 mm
- net +3V3: track 142.4 -> 149.0 mm
- net Net-(Q5-Pad1): track 0.00 -> 2.08 mm
- net Net-(Q6-Pad1): track 0.00 -> 2.04 mm
- net GND: vias 173 -> 159
Other:
- board text added: "24V 5V 3V3"
- board text added: "PCBrs - Teensy 4.1"
- board text removed: "PCBrs"

Commit message: update
Routing:
- net GND: track 1.36 -> 5.76 mm, vias 159 -> 162
- net /CANL: track 44.2 -> 40.2 mm
- net /S3_G: track 14.7 -> 12.7 mm
