File: PCB_Principal_V4/PCB_Principal_V4.kicad_sch (KiCad schematic)
At the start: 48 parts, among them J1 CAN, J10 NEXTION, J2 ENCODEUR_G, J3 ENCODEUR_D, J4 FAN, J5 CAN, J6 MOTOR_D, J7 BATT, J8 FAN, J9 MOTOR_G, Q1 Q_NPN_BEC, Q2 Q_NPN_BEC, U1 4504, U2 SN65HVD232, U3 TEENSY 4.1

Commit message: update last PCBs
Parts:
- added D7, D8: 1N4148W, Diode_SMD:D_SOD-123, symbol Diode:1N4148W
- added J11, J12: FAN, AREA_lib_Connector:Wuerth_2.54mm_2pins_61900211121, symbol Connector:Conn_01x02_Male
- added Q5, Q6: Q_NPN_BEC, Package_TO_SOT_SMD:SOT-23, symbol Device:Q_NPN_BEC
- added R11, R12: 10k, Resistor_SMD:R_0805_2012Metric_Pad1.20x1.40mm_HandSolder, symbol Device:R
Connections:
- net +24V: now also D7.1 (K), D8.1 (K), J11.1 (Pin_1), J12.1 (Pin_1)
- net GND: now also Q5.2 (E), Q6.2 (E)
- net PWM_FAN4: now reaches U3.29 (TX7)
- net PWM_FAN4: now also R12.1
- net PWM_FAN3: now reaches U3.30 (CRX3)
- net PWM_FAN3: now also R11.1
- new net: D7.2 (A), J11.2 (Pin_2), Q5.3 (C)
- new net: D8.2 (A), J12.2 (Pin_2), Q6.3 (C)
- new net: Q6.1 (B), R12.2
- new net: Q5.1 (B), R11.2
Other:
- moved on the sheet: D1, D5, H1, H2, H3, H4, J4, J8, Q1, Q2, R1, R2

Commit message: update
Parts:
- Q1, Q2, Q5, Q6: value Q_NPN_BEC -> SI2302S; symbol Device:Q_NPN_BEC -> Device:Q_NMOS_GSD
Changed lines of the file:
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@@
     (pin "2")
   )
-  (symbol (lib_id "Device:Q_NPN_BEC") (at 39.37 185.42 0) (unit 1)
+  (symbol (lib_id "Device:Q_NMOS_GSD") (at 39.37 185.42 0) (unit 1)
     (in_bom yes) (on_board yes) (fields_autoplaced)
     (property "Reference" "Q1" (id 0) (at 44.2214 184.5853 0)
       (effects (font (size 1.27 1.27)) (justify left))
     )
-    (property "Value" "Q_NPN_BEC" (id 1) (at 44.2214 187.1222 0)
+    (property "Value" "SI2302S " (id 1) (at 44.2214 187.1222 0)
       (effects (font (size 1.27 1.27)) (justify left))
     )
@@
     (pin "1")
   )
-  (symbol (lib_id "Device:Q_NPN_BEC") (at 78.74 185.42 0) (unit 1)
+  (symbol (lib_id "Device:Q_NMOS_GSD") (at 78.74 185.42 0) (unit 1)
     (in_bom yes) (on_board yes) (fields_autoplaced)
     (property "Reference" "Q2" (id 0) (at 83.5914 184.5853 0)
       (effects (font (size 1.27 1.27)) (justify left))
     )
-    (property "Value" "Q_NPN_BEC" (id 1) (at 83.5914 187.1222 0)
+    (property "Value" "SI2302S " (id 1) (at 83.5914 187.1222 0)
       (effects (font (size 1.27 1.27)) (justify left))
     )
@@
     (pin "1")
   )
-  (symbol (lib_id "Device:Q_NPN_BEC") (at 115.57 185.42 0) (unit 1)
+  (symbol (lib_id "Device:Q_NMOS_GSD") (at 115.57 185.42 0) (unit 1)
     (in_bom yes) (on_board yes) (fields_autoplaced)
     (property "Reference" "Q5" (id 0) (at 120.4214 184.5853 0)
       (effects (font (size 1.27 1.27)) (justify left))
     )
-    (property "Value" "Q_NPN_BEC" (id 1) (at 120.4214 187.1222 0)
+    (property "Value" "SI2302S " (id 1) (at 120.4214 187.1222 0)
       (effects (font (size 1.27 1.27)) (justify left))
     )
@@
     (pin "1")
   )
-  (symbol (lib_id "Device:Q_NPN_BEC") (at 154.94 185.42 0) (unit 1)
+  (symbol (lib_id "Device:Q_NMOS_GSD") (at 154.94 185.42 0) (unit 1)
     (in_bom yes) (on_board yes) (fields_autoplaced)
     (property "Reference" "Q6" (id 0) (at 159.7914 184.5853 0)
       (effects (font (size 1.27 1.27)) (justify left))
     )
-    (property "Value" "Q_NPN_BEC" (id 1) (at 159.7914 187.1222 0)
+    (property "Value" "SI2302S " (id 1) (at 159.7914 187.1222 0)
       (effects (font (size 1.27 1.27)) (justify left))
     )
@@
     )
     (path "/02879dbe-eeb5-4a9a-a50e-ab49eebaa379"
-      (reference "Q1") (unit 1) (value "Q_NPN_BEC") (footprint "Package_TO_SOT_SMD:SOT-23")
+      (reference "Q1") (unit 1) (value "SI2302S ") (footprint "Package_TO_SOT_SMD:SOT-23")
     )
     (path "/0d525ad4-3f7e-4e8e-b572-5aed774da48c"
-      (reference "Q2") (unit 1) (value "Q_NPN_BEC") (footprint "Package_TO_SOT_SMD:SOT-23")
+      (reference "Q2") (unit 1) (value "SI2302S ") (footprint "Package_TO_SOT_SMD:SOT-23")
     )
     (path "/59739e5e-6177-4c9f-b020-cdc056197113/00000000-0000-0000-0000-000062128337"
@@
     )
     (path "/917fb16e-24a9-435b-9f9c-44e17fc17a4a"
-      (reference "Q5") (unit 1) (value "Q_NPN_BEC") (footprint "Package_TO_SOT_SMD:SOT-23")
+      (reference "Q5") (unit 1) (value "SI2302S ") (footprint "Package_TO_SOT_SMD:SOT-23")
     )
     (path "/ea3b1909-42d0-4ff7-8a70-1794c5b61ac2"
-      (reference "Q6") (unit 1) (value "Q_NPN_BEC") (footprint "Package_TO_SOT_SMD:SOT-23")
+      (reference "Q6") (unit 1) (value "SI2302S ") (footprint "Package_TO_SOT_SMD:SOT-23")
     )
     (path "/3081c45f-0a62-4dc8-a706-c2b3c5e194d8"
