File: Carte_Alim_V7/Carte_Alim_V6_2022.kicad_sch (KiCad schematic)
At the start: 49 parts, among them J1 BAT_IN, J10 12VC, J11 12VC, J12 12VC, J13 12VP, J14 12VP, J15 12VP, J16 12VP, J17 12VP, J18 12VP, J19 5VC, J2 BAT_IN, J20 5V_CAN, J21 5VC, J22 5V_CAN, J23 5VC, J24 5V_CAN, J25 5VC, J26 5V_CAN, J27 5VP, J28 5VP, J29 5VP, J3 MOT_OUT, J30 5VP, J31 5VP, J32 5VP, J4 MOT_OUT, J5 MOT_OUT, J6 MOT_OUT, J7 12VC, J8 12VC, J9 12VC

Commit message: update last PCBs
Parts:
- removed D4, D7: LED, LED_SMD:LED_0805_2012Metric_Pad1.15x1.40mm_HandSolder, symbol Device:LED
- removed J10, J11, J12, J7, J8, J9: 12VC, AREA_lib_Connector:Wuerth_2.54mm_2pins_61900211121, symbol Connector:Conn_01x02_Male
- removed J19, J21, J23, J25: 5VC, AREA_lib_Connector:Wuerth_2.54mm_2pins_61900211121, symbol Connector:Conn_01x02_Male
- removed PS1, PS2: TSR_2-2450, AREA_lib_composant:CONV_TSR_2-2450, symbol AREA_composant:TSR_2-2450
- removed R12: 5.1K, Resistor_SMD:R_0805_2012Metric_Pad1.20x1.40mm_HandSolder, symbol Device:R
- removed R14: 560, Resistor_SMD:R_0805_2012Metric_Pad1.20x1.40mm_HandSolder, symbol Device:R
- D1, D3, D5: footprint LED_SMD:LED_0805_2012Metric_Pad1.15x1.40mm_HandSolder -> LED_SMD:LED_0805_2012Metric
- R1, R11, R13: footprint Resistor_SMD:R_0805_2012Metric_Pad1.20x1.40mm_HandSolder -> Resistor_SMD:R_0805_2012Metric
Other:
- note added: "Régulateur tension de commande 4A max"
- note added: "Sortie 5V CAN"
- note removed: "Régulateur tension de commande 2A max"
- note removed: "Sortie 12V/2A commande"
- note removed: "Sortie 5V/2A commande + CAN"
- moved on the sheet: D5, F1, J13, J14, J15, J16, J17, J18, J20, J22, J24, J26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
