File: Carte_Alim_V7/REGULO.kicad_sch (KiCad schematic)
At the start: 27 parts, among them U3 SIC466ED-T1-GE3

Commit message: update last PCBs
Parts:
- removed C49, C50, C51: 22u, Capacitor_SMD:C_1210_3225Metric_Pad1.33x2.70mm_HandSolder, symbol Device:C
- added C17, C24: 10u/50V, Capacitor_SMD:CP_Elec_5x5.4, symbol Device:C_Polarized
- added C25: 330u/25V, Capacitor_SMD:CP_Elec_8x10.5, symbol Device:C_Polarized
- C35, C36, C41, C42, C43, C44, C45: footprint Capacitor_SMD:C_0805_2012Metric_Pad1.18x1.45mm_HandSolder -> Capacitor_SMD:C_0805_2012Metric
- C37: footprint Capacitor_SMD:C_1210_3225Metric_Pad1.33x2.70mm_HandSolder -> Capacitor_SMD:C_1206_3216Metric; Part (none) -> C3216X5R1V226MTJ00E
- C38, C46, C47, C48: footprint Capacitor_SMD:C_1210_3225Metric_Pad1.33x2.70mm_HandSolder -> Capacitor_SMD:C_1206_3216Metric
- D6: footprint LED_SMD:LED_0805_2012Metric_Pad1.15x1.40mm_HandSolder -> LED_SMD:LED_0805_2012Metric
- R22, R23, R24, R25, R26, R27, R28, R29, R30: footprint Resistor_SMD:R_0603_1608Metric_Pad0.98x0.95mm_HandSolder -> Resistor_SMD:R_0603_1608Metric
Connections:
- net GND: now also U3.30 (PGND), U3.A30 (PGND), C17.2, C24.2, C25.2; no longer U3.30.1 (PGND), U3.30.2 (PGND)
- net VIN: now also C17.1, C24.1
- net VOUT: now also C25.1
Other:
- note added: "1206"
- note added: "C3216X5R1V226MTJ00E"
- note removed: "1210"
- moved on the sheet: C35, C36, C37, C38

Commit message: update
Parts:
- renumbered C35 to C1, C44 to C10, C45 to C11, C46 to C12, C47 to C13, C48 to C14, C24 to C15, C25 to C16, C36 to C2, C37 to C3, C38 to C4, C17 to C5, C41 to C7, C42 to C8, C43 to C9, D6 to D2, L3 to L1, R30 to R10, R22 to R2, R23 to R3, R24 to R4, R25 to R5, R26 to R6, R27 to R7, R28 to R8, R29 to R9, U3 to U1
Changed lines of the file:
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@@
   (symbol (lib_id "Device:C") (at 231.14 57.15 0)
     (in_bom yes) (on_board yes)
-    (property "Reference" "C48" (id 0) (at 231.14 53.34 0)
+    (property "Reference" "C14" (id 0) (at 231.14 53.34 0)
       (effects (font (size 1.27 1.27)) (justify left))
     )
@@
   (symbol (lib_id "power:GND") (at 175.26 74.93 0)
     (in_bom yes) (on_board yes)
-    (property "Reference" "#PWR0101" (id 0) (at 175.26 81.28 0)
+    (property "Reference" "#PWR089" (id 0) (at 175.26 81.28 0)
       (effects (font (size 1.27 1.27)) hide)
     )
@@
   (symbol (lib_id "Carte_Alim_V5-rescue:SIC461ED-T1-GE3-AREA_composant") (at 146.05 54.61 0)
     (in_bom yes) (on_board yes)
-    (property "Reference" "U3" (id 0) (at 146.05 27.5082 0))
+    (property "Reference" "U1" (id 0) (at 146.05 27.5082 0))
     (property "Value" "SIC466ED-T1-GE3" (id 1) (at 146.05 29.8196 0))
     (property "Footprint" "AREA_lib_composant:SIC463EDT1GE3" (id 2) (at 146.05 54.61 0)
@@
     (pin "3")
     (pin "30")
-    (pin "A30")
     (pin "4")
     (pin "5")
@@
     (pin "8")
     (pin "9")
+    (pin "A30")
   )
   (symbol (lib_id "Device:C") (at 83.82 57.15 0)
     (in_bom yes) (on_board yes)
-    (property "Reference" "C38" (id 0) (at 83.82 54.61 0)
+    (property "Reference" "C4" (id 0) (at 83.82 54.61 0)
       (effects (font (size 1.27 1.27)) (justify left))
     )
@@
   (symbol (lib_id "Device:C") (at 96.52 57.15 0)
     (in_bom yes) (on_board yes)
-    (property "Reference" "C36" (id 0) (at 96.52 54.61 0)
+    (property "Reference" "C2" (id 0) (at 96.52 54.61 0)
       (effects (font (size 1.27 1.27)) (justify left))
     )
@@
   (symbol (lib_id "Device:C_Polarized") (at 236.22 57.15 0)
     (in_bom yes) (on_board yes) (fields_autoplaced)
-    (property "Reference" "C25" (id 0) (at 239.141 55.4263 0)
+    (property "Reference" "C16" (id 0) (at 239.141 55.4263 0)
       (effects (font (size 1.27 1.27)) (justify left))
     )
@@
   (symbol (lib_id "Device:R") (at 200.66 55.88 180)
     (in_bom yes) (on_board yes)
-    (property "Reference" "R29" (id 0) (at 200.66 57.15 90))
+    (property "Reference" "R9" (id 0) (at 200.66 57.15 90))
     (property "Value" "10k" (id 1) (at 204.47 54.61 0))
     (property "Footprint" "Resistor_SMD:R_0603_1608Metric" (id 2) (at 202.438 55.88 90)
@@
   (symbol (lib_id "Device:R") (at 113.03 54.61 0)
     (in_bom yes) (on_board yes)
-    (property "Reference" "R24" (id 0) (at 114.808 53.4416 0)
+    (property "Reference" "R4" (id 0) (at 114.808 53.4416 0)
       (effects (font (size 1.27 1.27)) (justify left))
     )
@@
   (symbol (lib_id "Device:R") (at 189.23 57.15 270)
     (in_bom yes) (on_board yes)
-    (property "Reference" "R27" (id 0) (at 187.96 57.15 90))
+    (property "Reference" "R7" (id 0) (at 187.96 57.15 90))
     (property "Value" "3.3" (id 1) (at 187.96 54.61 90))
     (property "Footprint" "Resistor_SMD:R_0603_1608Metric" (id 2) (at 189.23 55.372 90)
@@
   (symbol (lib_id "Device:C") (at 91.44 57.15 0)
     (in_bom yes) (on_board yes)
-    (property "Reference" "C35" (id 0) (at 91.44 54.61 0)
+    (property "Reference" "C1" (id 0) (at 91.44 54.61 0)
       (effects (font (size 1.27 1.27)) (justify left))
     )
@@
   (symbol (lib_id "Device:L") (at 182.88 41.91 90)
     (in_bom yes) (on_board yes)
-    (property "Reference" "L3" (id 0) (at 179.07 40.64 90))
+    (property "Reference" "L1" (id 0) (at 179.07 40.64 90))
     (property "Value" "4.7uH" (id 1) (at 187.96 40.64 90))
     (property "Footprint" "Inductor_SMD:L_Vishay_IHLP-6767" (id 2) (at 182.88 41.91 0)
@@
   (symbol (lib_id "Device:R") (at 119.38 68.58 0)
     (in_bom yes) (on_board yes)
-    (property "Reference" "R25" (id 0) (at 121.158 67.4116 0)
+    (property "Reference" "R5" (id 0) (at 121.158 67.4116 0)
       (effects (font (size 1.27 1.27)) (justify left))
     )
@@
   (symbol (lib_id "power:GND") (at 33.02 17.78 0)
     (in_bom yes) (on_board yes)
-    (property "Reference" "#PWR097" (id 0) (at 33.02 24.13 0)
+    (property "Reference" "#PWR085" (id 0) (at 33.02 24.13 0)
       (effects (font (size 1.27 1.27)) hide)
     )
@@
   (symbol (lib_id "Device:C") (at 78.74 57.15 0)
     (in_bom yes) (on_board yes)
-    (property "Reference" "C37" (id 0) (at 78.74 54.61 0)
+    (property "Reference" "C3" (id 0) (at 78.74 54.61 0)
       (effects (font (size 1.27 1.27)) (justify left))
     )
@@
   (symbol (lib_id "Device:C") (at 191.77 52.07 270)
     (in_bom yes) (on_board yes)
-    (property "Reference" "C44" (id 0) (at 193.04 50.8 90)
+    (property "Reference" "C10" (id 0) (at 193.04 50.8 90)
       (effects (font (size 1.27 1.27)) (justify left))
     )
@@
   (symbol (lib_id "Device:R") (at 107.95 66.04 0)
     (in_bom yes) (on_board yes)
-    (property "Reference" "R22" (id 0) (at 109.728 64.8716 0)
+    (property "Reference" "R2" (id 0) (at 109.728 64.8716 0)
       (effects (font (size 1.27 1.27)) (justify left))
     )
@@
   (symbol (lib_id "Device:C_Polarized") (at 58.42 57.15 0)
     (in_bom yes) (on_board yes)
-    (property "Reference" "C17" (id 0) (at 61.341 55.4263 0)
+    (property "Reference" "C5" (id 0) (at 61.341 55.4263 0)
       (effects (font (size 1.27 1.27)) (justify left))
     )
@@
   (symbol (lib_id "Device:R") (at 113.03 45.72 0)
     (in_bom yes) (on_board yes)
-    (property "Reference" "R23" (id 0) (at 114.808 44.5516 0)
+    (property "Reference" "R3" (id 0) (at 114.808 44.5516 0)
       (effects (font (size 1.27 1.27)) (justify left))
     )
@@
   (symbol (lib_id "Device:C_Polarized") (at 68.58 57.15 0)
     (in_bom yes) (on_board yes)
-    (property "Reference" "C24" (id 0) (at 71.501 55.4263 0)
+    (property "Reference" "C15" (id 0) (at 71.501 55.4263 0)
       (effects (font (size 1.27 1.27)) (justify left))
     )
@@
   (symbol (lib_id "Device:R") (at 252.73 57.15 0)
     (in_bom yes) (on_board yes)
-    (property "Reference" "R30" (id 0) (at 254.508 55.9816 0)
+    (property "Reference" "R10" (id 0) (at 254.508 55.9816 0)
       (effects (font (size 1.27 1.27)) (justify left))
     )
@@
   (symbol (lib_id "Device:C") (at 179.07 57.15 270)
     (in_bom yes) (on_board yes)
-    (property "Reference" "C42" (id 0) (at 180.34 55.88 90)
+    (property "Reference" "C8" (id 0) (at 180.34 55.88 90)
       (effects (font (size 1.27 1.27)) (justify left))
     )
@@
   (symbol (lib_id "power:GND") (at 107.95 78.74 0)
     (in_bom yes) (on_board yes)
-    (property "Reference" "#PWR0100" (id 0) (at 107.95 85.09 0)
+    (property "Reference" "#PWR088" (id 0) (at 107.95 85.09 0)
       (effects (font (size 1.27 1.27)) hide)
     )
@@
   (symbol (lib_id "Device:C") (at 208.28 57.15 0)
     (in_bom yes) (on_board yes)
-    (property "Reference" "C45" (id 0) (at 208.28 54.61 0)
+    (property "Reference" "C11" (id 0) (at 208.28 54.61 0)
       (effects (font (size 1.27 1.27)) (justify left))
     )
@@
   (symbol (lib_id "Device:R") (at 200.66 45.72 180)
     (in_bom yes) (on_board yes)
-    (property "Reference" "R28" (id 0) (at 200.66 46.99 90))
+    (property "Reference" "R8" (id 0) (at 200.66 46.99 90))
     (property "Value" "52.3k" (id 1) (at 204.47 44.45 0))
     (property "Footprint" "Resistor_SMD:R_0603_1608Metric" (id 2) (at 202.438 45.72 90)
@@
   (symbol (lib_id "Device:C") (at 220.98 57.15 0)
     (in_bom yes) (on_board yes)
-    (property "Reference" "C46" (id 0) (at 220.98 53.34 0)
+    (property "Reference" "C12" (id 0) (at 220.98 53.34 0)
       (effects (font (size 1.27 1.27)) (justify left))
     )
@@
   (symbol (lib_id "Device:C") (at 184.15 34.29 270)
     (in_bom yes) (on_board yes)
-    (property "Reference" "C43" (id 0) (at 185.42 33.02 90)
+    (property "Reference" "C9" (id 0) (at 185.42 33.02 90)
       (effects (font (size 1.27 1.27)) (justify left))
     )
@@
   (symbol (lib_id "Device:R") (at 176.53 52.07 270)
     (in_bom yes) (on_board yes)
-    (property "Reference" "R26" (id 0) (at 175.26 52.07 90))
+    (property "Reference" "R6" (id 0) (at 175.26 52.07 90))
     (property "Value" "100k" (id 1) (at 181.61 53.34 90))
     (property "Footprint" "Resistor_SMD:R_0603_1608Metric" (id 2) (at 176.53 50.292 90)
@@
   (symbol (lib_id "Device:C") (at 226.06 57.15 0)
     (in_bom yes) (on_board yes)
-    (property "Reference" "C47" (id 0) (at 226.06 53.34 0)
+    (property "Reference" "C13" (id 0) (at 226.06 53.34 0)
       (effects (font (size 1.27 1.27)) (justify left))
     )
@@
   (symbol (lib_id "power:GND") (at 194.31 34.29 0)
     (in_bom yes) (on_board yes)
-    (property "Reference" "#PWR0102" (id 0) (at 194.31 40.64 0)
+    (property "Reference" "#PWR090" (id 0) (at 194.31 40.64 0)
       (effects (font (size 1.27 1.27)) hide)
     )
@@
   (symbol (lib_id "Device:C") (at 114.3 67.31 0)
     (in_bom yes) (on_board yes)
-    (property "Reference" "C41" (id 0) (at 114.3 64.77 0)
+    (property "Reference" "C7" (id 0) (at 114.3 64.77 0)
       (effects (font (size 1.27 1.27)) (justify left))
     )
@@
   (symbol (lib_id "Device:LED") (at 252.73 68.58 90)
     (in_bom yes) (on_board yes)
-    (property "Reference" "D6" (id 0) (at 255.7272 67.5894 90)
+    (property "Reference" "D2" (id 0) (at 255.7272 67.5894 90)
       (effects (font (size 1.27 1.27)) (justify right))
     )
