File: Carte_Alim_V7/REGULO5v.kicad_sch (KiCad schematic)
At the start: 13 parts, among them U2 TPS5450ddar

Commit message: update last PCBs
Parts:
- removed C5: 100n, Capacitor_SMD:C_0805_2012Metric_Pad1.18x1.45mm_HandSolder, symbol Device:C
- added C26, C27: 10u/50V, Capacitor_SMD:CP_Elec_5x5.4, symbol Device:C_Polarized
- C18, C19: value 10u -> 22u; footprint Capacitor_SMD:C_1210_3225Metric_Pad1.33x2.70mm_HandSolder -> Capacitor_SMD:C_1206_3216Metric
- C20, C22, C23, C6: footprint Capacitor_SMD:C_0805_2012Metric_Pad1.18x1.45mm_HandSolder -> Capacitor_SMD:C_0805_2012Metric
- D8: footprint Diode_SMD:D_SMC_Handsoldering -> Diode_SMD:D_SMC
- L2: footprint Inductor_SMD:L_Wuerth_HCI-1335 -> Inductor_SMD:L_Wuerth_HCI-1030
- R15, R16: footprint Resistor_SMD:R_0603_1608Metric_Pad0.98x0.95mm_HandSolder -> Resistor_SMD:R_0603_1608Metric
Connections:
- net GND: now also C26.2, C27.2
- net VIN: now also C26.1, C27.1
Other:
- note added: "same ref as previous 22u"
- moved on the sheet: C18, C19, C6

Commit message: update
Parts:
- added F2: 3557-2, AREA_lib_composant:FUSE_3557-2, symbol AREA_composant:3557-2
- C21: value 330u -> 220u
Connections:
- net VOUT: now also F2.3; no longer C21.1, C22.1, C23.1, L2.2, R15.1
- new net: C21.1, C22.1, C23.1, F2.1, L2.2, R15.1
Changed lines of the file:
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@@
-    (stroke (width 0) (type default) (color 0 0 0 0))
-  )
-  (wire (pts (xy 187.96 41.91) (xy 199.39 41.91))
     (stroke (width 0) (type default) (color 0 0 0 0))
   )
@@
   )
   (wire (pts (xy 134.62 41.91) (xy 146.05 41.91))
+    (stroke (width 0) (type default) (color 0 0 0 0))
+  )
+  (wire (pts (xy 187.96 41.91) (xy 190.5 41.91))
+    (stroke (width 0) (type default) (color 0 0 0 0))
+  )
+  (wire (pts (xy 200.66 41.91) (xy 203.2 41.91))
     (stroke (width 0) (type default) (color 0 0 0 0))
   )
@@
     (effects (font (size 1.27 1.27)) (justify right))
   )
-  (hierarchical_label "VOUT" (shape output) (at 198.12 41.91 0)
+  (hierarchical_label "VOUT" (shape output) (at 203.2 41.91 0)
     (effects (font (size 1.27 1.27)) (justify left))
   )
@@
       (effects (font (size 1.27 1.27)) (justify left))
     )
-    (property "Value" "330u" (id 1) (at 161.29 53.34 0)
+    (property "Value" "220u" (id 1) (at 161.29 53.34 0)
       (effects (font (size 1.27 1.27)) (justify left))
     )
@@
     (pin "2")
   )
+  (symbol (lib_id "AREA_composant:3557-2") (at 195.58 41.91 0) (unit 1)
+    (in_bom yes) (on_board yes)
+    (property "Reference" "F2" (id 0) (at 195.58 39.37 0))
+    (property "Value" "3557-2" (id 1) (at 195.58 44.45 0))
+    (property "Footprint" "AREA_lib_composant:FUSE_3557-2" (id 2) (at 195.58 41.91 0)
+      (effects (font (size 1.27 1.27)) (justify left bottom) hide)
+    )
+    (property "Datasheet" "" (id 3) (at 195.58 41.91 0)
+      (effects (font (size 1.27 1.27)) (justify left bottom) hide)
+    )
+    (property "MANUFACTURER" "KEYSTONE" (id 4) (at 195.58 41.91 0)
+      (effects (font (size 1.27 1.27)) (justify left bottom) hide)
+    )
+    (pin "1")
+    (pin "2")
+    (pin "3")
+    (pin "4")
+  )
   (symbol (lib_id "Device:C") (at 93.98 53.34 0) (unit 1)
