File: PCB_CAN_sortie/PCB_CAN_sortie.kicad_pcb (KiCad board)
At the start: 2 copper layers, 27.5 x 27.5 mm, 6 parts, among them J1 CAN, J2 CAN

Commit message: lots of stuf
Other:
- net class Default removed
