File: PCB_stepper/PCB_stepper.kicad_sch (KiCad schematic)
At the start: 47 parts, among them J1 USB_C_Receptacle_USB2.0, J2 CON_CAN, J3 CON_CAN, J4 12V, J5 Conn_01x04_Male, SW1 RST, SW2 BOOT, U1 STM32F302C6Tx, U2 SN65HVD232, U3 NCP1117-3.3_SOT223, Y1 8MHz

Commit message: MAJ principal + stepper
Parts:
- C14: footprint Capacitor_THT:CP_Radial_D5.0mm_P2.00mm -> Capacitor_SMD:CP_Elec_5x5.4
- C15: value 100u -> 47u; footprint Capacitor_THT:CP_Radial_D8.0mm_P3.50mm -> Capacitor_SMD:CP_Elec_6.3x5.4
- C6: value 0.1u -> 100n
Connections:
- net +3V3: no longer C14.1
- net +5V: now also C14.1
- net EN: now also U1.19 (PB1); no longer U1.30 (PA9)
- net M0: now also U1.18 (PB0); no longer U1.29 (PA8)
- net at U1.25 (PB12): no longer D1.2 (A)
- net USR_LED: now reaches U1.43 (PB7)
- net USR_LED: now also D1.2 (A)
- net USART3_RX: no longer names the net of U1.22 (PB11)
- net USART3_TX: no longer names the net of U1.21 (PB10)
Other:
- moved on the sheet: C1, C10, C2, C5, C7, C9, D1, R1

Commit message: update
Parts:
- added R10, R11, R12: 10k, Resistor_SMD:R_0805_2012Metric, symbol Device:R
- added SW3: SW_DIP_x03, Button_Switch_SMD:SW_DIP_SPSTx03_Slide_KingTek_DSHP03TJ_W5.25mm_P1.27mm_JPin, symbol Switch:SW_DIP_x03
- C1, C10, C11, C12, C16, C17, C2, C3, C4, C5, C6, C7, C8, C9: footprint Capacitor_SMD:C_0805_2012Metric_Pad1.18x1.45mm_HandSolder -> Capacitor_SMD:C_0805_2012Metric
- D3, D4, D5: footprint LED_SMD:LED_0805_2012Metric_Pad1.15x1.40mm_HandSolder -> LED_SMD:LED_0805_2012Metric
- R1, R2, R3, R4, R5, R6, R7, R8, R9: footprint Resistor_SMD:R_0805_2012Metric_Pad1.20x1.40mm_HandSolder -> Resistor_SMD:R_0805_2012Metric
Connections:
- net +3V3: now also SW3.1, SW3.2, SW3.3
- net GND: now also R10.1, R11.1, R12.1
- net at U1.26 (PB13): now also R10.2, SW3.6
- net at U1.27 (PB14): now also R11.2, SW3.5
- net at U1.28 (PB15): now also R12.2, SW3.4
Other:
- moved on the sheet: R2, SW2
